Commit message: Update joint names.

File: robotiq_description/urdf/robotiq_sim_gripper.ros2_control.xacro (robot description, xacro)
@@ -12,27 +12,6 @@
                 <state_interface name="velocity"/>
             </joint>
-            <joint name="right_outer_knuckle_joint">
-                <param name="mimic">finger_joint</param>
-                <param name="multiplier">1</param>
-                <command_interface name="position"/>
-                <state_interface name="position"/>
-                <state_interface name="velocity"/>
-            </joint>
-            <joint name="right_inner_knuckle_joint">
-                <param name="mimic">finger_joint</param>
-                <param name="multiplier">1</param>
-                <command_interface name="position"/>
-                <state_interface name="position"/>
-                <state_interface name="velocity"/>
-            </joint>
-            <joint name="left_inner_knuckle_joint">
-                <param name="mimic">finger_joint</param>
-                <param name="multiplier">1</param>
-                <command_interface name="position"/>
-                <state_interface name="position"/>
-                <state_interface name="velocity"/>
-            </joint>
-            <joint name="left_inner_finger_joint">
-                <param name="mimic">finger_joint</param>
+            <joint name="robotiq_85_right_knuckle_joint">
+                <param name="mimic">robotiq_85_left_knuckle_joint</param>
                 <param name="multiplier">-1</param>
                 <command_interface name="position"/>
@@ -40,10 +19,31 @@
                 <state_interface name="velocity"/>
             </joint>
-            <joint name="right_inner_finger_joint">
-                <param name="mimic">finger_joint</param>
+            <joint name="robotiq_85_left_inner_knuckle_joint">
+                <param name="mimic">robotiq_85_left_knuckle_joint</param>
+                <param name="multiplier">1</param>
+                <command_interface name="position" />
+                <state_interface name="position" />
+                <state_interface name="velocity" />
+            </joint>
+            <joint name="robotiq_85_right_inner_knuckle_joint">
+                <param name="mimic">robotiq_85_left_knuckle_joint</param>
                 <param name="multiplier">-1</param>
-                <command_interface name="position"/>
-                <state_interface name="position"/>
-                <state_interface name="velocity"/>
+                <command_interface name="position" />
+                <state_interface name="position" />
+                <state_interface name="velocity" />
+            </joint>
+            <joint name="robotiq_85_left_finger_tip_joint">
+                <param name="mimic">robotiq_85_left_knuckle_joint</param>
+                <param name="multiplier">-1</param>
+                <command_interface name="position" />
+                <state_interface name="position" />
+                <state_interface name="velocity" />
+            </joint>
+            <joint name="robotiq_85_right_finger_tip_joint">
+                <param name="mimic">robotiq_85_left_knuckle_joint</param>
+                <param name="multiplier">1</param>
+                <command_interface name="position" />
+                <state_interface name="position" />
+                <state_interface name="velocity" />
             </joint>
         </ros2_control>

Commit message: Add sim_isaac ros2_control xacro arg

File: robotiq_description/urdf/robotiq_sim_gripper.ros2_control.xacro (robot description, xacro)
@@ -1,8 +1,20 @@
 <?xml version="1.0"?>
 <robot xmlns:xacro="http://www.ros.org/wiki/xacro">
-    <xacro:macro name="robotiq_sim_gripper_ros2_control" params="name">
+    <xacro:macro name="robotiq_sim_gripper_ros2_control" params="
+      name
+      sim_isaac:=false
+      use_fake_hardware:=false">
         <ros2_control name="${name}" type="system">
             <hardware>
-                <plugin>fake_components/GenericSystem</plugin>
+                <xacro:if value="${sim_isaac}">
+                    <plugin>isaac_ros2_control/IsaacSystem</plugin>
+                    <param name="joint_commands_topic">/isaac_joint_commands</param>
+                    <param name="joint_states_topic">/isaac_joint_states</param>
+                </xacro:if>
+                <xacro:if value="${use_fake_hardware}">
+                    <plugin>mock_components/GenericSystem</plugin>
+                    <param name="fake_sensor_commands">${fake_sensor_commands}</param>
+                    <param name="state_following_offset">0.0</param>
+                </xacro:if>
             </hardware>
             <joint name="robotiq_85_left_knuckle_joint">

Commit message: Fixes after testing

File: robotiq_description/urdf/robotiq_sim_gripper.ros2_control.xacro (robot description, xacro)
@@ -1,9 +1,6 @@
 <?xml version="1.0"?>
 <robot xmlns:xacro="http://www.ros.org/wiki/xacro">
-    <xacro:macro name="robotiq_sim_gripper_ros2_control" params="
-      name
-      sim_ignition:=false
-      sim_isaac:=false
-      use_fake_hardware:=false">
+    <xacro:macro name="robotiq_sim_gripper_ros2_control"
+                 params="name sim_ignition:=false sim_isaac:=false use_fake_hardware:=false">
         <ros2_control name="${name}" type="system">
             <hardware>
@@ -13,11 +10,9 @@
                     <param name="joint_states_topic">/isaac_joint_states</param>
                 </xacro:if>
+                <xacro:if value="${sim_ignition}">
+                    <plugin>ign_ros2_control/IgnitionSystem</plugin>
+                </xacro:if>
                 <xacro:if value="${use_fake_hardware}">
-                    <xacro:if value="${sim_ignition}">
-                        <plugin>ign_ros2_control/IgnitionSystem</plugin>
-                    </xacro:if>
-                    <xacro:unless value="${sim_ignition}">
-                        <plugin>mock_components/GenericSystem</plugin>
-                    </xacro:unless>
+                    <plugin>mock_components/GenericSystem</plugin>
                     <param name="fake_sensor_commands">${fake_sensor_commands}</param>
                     <param name="state_following_offset">0.0</param>
@@ -27,11 +22,13 @@
                 <!-- With Ignition, we have mimic joints, so we only need this command interface activated -->
                 <xacro:if value="${sim_ignition}">
-                    <param name="initial_position">0.2</param>
+                    <state_interface name="position">
+                        <param name="initial_value">0.2</param>
+                    </state_interface>
                 </xacro:if>
                 <xacro:unless value="${sim_ignition}">
                     <param name="initial_position">0.7929</param>
+                    <state_interface name="position"/>
                 </xacro:unless>
                 <command_interface name="position" />
-                <state_interface name="position"/>
                 <state_interface name="velocity"/>
             </joint>
@@ -81,5 +78,4 @@
                 </xacro:unless>
             </joint>
-            <!-- Not active for Ignition -->
             <xacro:unless value="${sim_ignition}">
                 <gpio name="reactivate_gripper">

Commit message: Add Ignition Gazebo switches to ROS2 control sim config (#8)
* Add Ignition Gazebo switches to ROS2 control sim config

* Fixes after testing

* PR comments

File: robotiq_description/urdf/robotiq_sim_gripper.ros2_control.xacro (robot description, xacro)
@@ -1,9 +1,8 @@
 <?xml version="1.0"?>
 <robot xmlns:xacro="http://www.ros.org/wiki/xacro">
-    <xacro:macro name="robotiq_sim_gripper_ros2_control" params="
-      name
-      sim_isaac:=false
-      use_fake_hardware:=false">
+    <xacro:macro name="robotiq_sim_gripper_ros2_control"
+                 params="name sim_ignition:=false sim_isaac:=false use_fake_hardware:=true">
         <ros2_control name="${name}" type="system">
+            <!-- Plugins -->
             <hardware>
                 <xacro:if value="${sim_isaac}">
@@ -11,4 +10,7 @@
                     <param name="joint_commands_topic">/isaac_joint_commands</param>
                     <param name="joint_states_topic">/isaac_joint_states</param>
+                </xacro:if>
+                <xacro:if value="${sim_ignition}">
+                    <plugin>ign_ros2_control/IgnitionSystem</plugin>
                 </xacro:if>
                 <xacro:if value="${use_fake_hardware}">
@@ -18,8 +20,17 @@
                 </xacro:if>
             </hardware>
+            <!-- Joint interfaces -->
             <joint name="robotiq_85_left_knuckle_joint">
-                <param name="initial_position">0.7929</param>
+                <!-- With Ignition, we have mimic joints, so we only need this command interface activated -->
+                <xacro:if value="${sim_ignition}">
+                    <state_interface name="position">
+                        <param name="initial_value">0.2</param>
+                    </state_interface>
+                </xacro:if>
+                <xacro:unless value="${sim_ignition}">
+                    <param name="initial_position">0.7929</param>
+                    <state_interface name="position"/>
+                </xacro:unless>
                 <command_interface name="position" />
-                <state_interface name="position"/>
                 <state_interface name="velocity"/>
             </joint>
@@ -27,40 +38,53 @@
                 <param name="mimic">robotiq_85_left_knuckle_joint</param>
                 <param name="multiplier">-1</param>
-                <command_interface name="position"/>
-                <state_interface name="position"/>
-                <state_interface name="velocity"/>
+                <xacro:unless value="${sim_ignition}">
+                    <command_interface name="position"/>
+                    <state_interface name="position"/>
+                    <state_interface name="velocity"/>
+                </xacro:unless>
             </joint>
             <joint name="robotiq_85_left_inner_knuckle_joint">
                 <param name="mimic">robotiq_85_left_knuckle_joint</param>
                 <param name="multiplier">1</param>
-                <command_interface name="position" />
-                <state_interface name="position" />
-                <state_interface name="velocity" />
+                <xacro:unless value="${sim_ignition}">
+                    <command_interface name="position"/>
+                    <state_interface name="position"/>
+                    <state_interface name="velocity"/>
+                </xacro:unless>
             </joint>
             <joint name="robotiq_85_right_inner_knuckle_joint">
                 <param name="mimic">robotiq_85_left_knuckle_joint</param>
                 <param name="multiplier">-1</param>
-                <command_interface name="position" />
-                <state_interface name="position" />
-                <state_interface name="velocity" />
+                <xacro:unless value="${sim_ignition}">
+                    <command_interface name="position"/>
+                    <state_interface name="position"/>
+                    <state_interface name="velocity"/>
+                </xacro:unless>
             </joint>
             <joint name="robotiq_85_left_finger_tip_joint">
                 <param name="mimic">robotiq_85_left_knuckle_joint</param>
                 <param name="multiplier">-1</param>
-                <command_interface name="position" />
-                <state_interface name="position" />
-                <state_interface name="velocity" />
+                <xacro:unless value="${sim_ignition}">
+                    <command_interface name="position"/>
+                    <state_interface name="position"/>
+                    <state_interface name="velocity"/>
+                </xacro:unless>
             </joint>
             <joint name="robotiq_85_right_finger_tip_joint">
                 <param name="mimic">robotiq_85_left_knuckle_joint</param>
                 <param name="multiplier">1</param>
-                <command_interface name="position" />
-                <state_interface name="position" />
-                <state_interface name="velocity" />
+                <xacro:unless value="${sim_ignition}">
+                    <command_interface name="position"/>
+                    <state_interface name="position"/>
+                    <state_interface name="velocity"/>
+                </xacro:unless>
             </joint>
-            <gpio name="reactivate_gripper">
-                <command_interface name="reactivate_gripper_cmd" />
-                <command_interface name="reactivate_gripper_response" />
-            </gpio>
+            <!-- Only add this with fake hardware mode -->
+            <xacro:unless value="${sim_ignition or sim_isaac}">
+                <gpio name="reactivate_gripper">
+                    <command_interface name="reactivate_gripper_cmd" />
+                    <command_interface name="reactivate_gripper_response" />
+                </gpio>
+            </xacro:unless>
         </ros2_control>
     </xacro:macro>
