Commit message: Add com_port parameter.

File: robotiq_description/urdf/robotiq_gripper.ros2_control.xacro (robot description, xacro)
@@ -1,10 +1,10 @@
 <?xml version="1.0"?>
 <robot xmlns:xacro="http://www.ros.org/wiki/xacro">
-    <xacro:macro name="robotiq_gripper_ros2_control" params="name">
+    <xacro:macro name="robotiq_gripper_ros2_control" params="name com_port">
         <ros2_control name="${name}" type="actuator">
             <hardware>
                 <plugin>robotiq_driver/RobotiqGripperHardwareInterface</plugin>
                 <param name="gripper_closed_position">0.7929</param>
-                <param name="COM_port">/dev/ttyUSB0</param>
+                <param name="COM_port">${com_port}</param>
                 <param name="gripper_speed_multiplier">1.0</param>
                 <param name="gripper_force_multiplier">0.5</param>

Commit message: Update joint name.

File: robotiq_description/urdf/robotiq_gripper.ros2_control.xacro (robot description, xacro)
@@ -10,5 +10,5 @@
                 <param name="gripper_force_multiplier">0.5</param>
             </hardware>
-            <joint name="robotiq_85_left_knuckle_joint">
+            <joint name="finger_joint">
                 <param name="initial_position">0.7929</param>
                 <command_interface name="position" />

Commit message: Add gripper URDF.

File: robotiq_description/urdf/robotiq_gripper.ros2_control.xacro (robot description, xacro)
@@ -10,5 +10,5 @@
                 <param name="gripper_force_multiplier">0.5</param>
             </hardware>
-            <joint name="finger_joint">
+            <joint name="robotiq_85_left_knuckle_joint">
                 <param name="initial_position">0.7929</param>
                 <command_interface name="position" />

Commit message: Unify urdf files.

File: robotiq_description/urdf/robotiq_gripper.ros2_control.xacro (robot description, xacro)
@@ -1,20 +1,86 @@
 <?xml version="1.0"?>
 <robot xmlns:xacro="http://www.ros.org/wiki/xacro">
-    <xacro:macro name="robotiq_gripper_ros2_control" params="name com_port">
-        <ros2_control name="${name}" type="actuator">
-            <hardware>
-                <plugin>robotiq_driver/RobotiqGripperHardwareInterface</plugin>
-                <param name="gripper_closed_position">0.7929</param>
-                <param name="COM_port">${com_port}</param>
-                <param name="gripper_speed_multiplier">1.0</param>
-                <param name="gripper_force_multiplier">0.5</param>
-            </hardware>
-            <joint name="robotiq_85_left_knuckle_joint">
-                <param name="initial_position">0.7929</param>
-                <command_interface name="position" />
-                <state_interface name="position" />
-                <state_interface name="velocity" />
-            </joint>
-        </ros2_control>
+    <xacro:macro name="robotiq_gripper_ros2_control" params="name com_port use_fake_hardware:=false sim_gz:=false">
+        <!-- ros2_control custom hardware interface -->
+        <xacro:unless value="${use_fake_hardware or sim_gz}">
+            <ros2_control name="${name}" type="actuator">
+                <hardware>
+                    <plugin>robotiq_driver/RobotiqGripperHardwareInterface</plugin>
+                    <param name="gripper_closed_position">0.7929</param>
+                    <param name="COM_port">${com_port}</param>
+                    <param name="gripper_speed_multiplier">1.0</param>
+                    <param name="gripper_force_multiplier">0.5</param>
+                </hardware>
+                <joint name="robotiq_85_left_knuckle_joint">
+                    <param name="initial_position">0.7929</param>
+                    <command_interface name="position" />
+                    <state_interface name="position" />
+                    <state_interface name="velocity" />
+                </joint>
+            </ros2_control>
+        </xacro:unless>
+        <xacro:if value="${use_fake_hardware or sim_gz}">
+            <ros2_control name="${name}" type="system">
+                <hardware>
+                    <!-- ros2_control fake component -->
+                    <xacro:if value="${use_fake_hardware}">
+                        <plugin>fake_components/GenericSystem</plugin>
+                    </xacro:if>
+                    <!-- gz simulation -->
+                    <xacro:if value="${sim_gz}">
+                        <plugin>ign_ros2_control/IgnitionSystem</plugin>
+                    </xacro:if>
+                </hardware>
+                <joint name="robotiq_85_left_knuckle_joint">
+                    <param name="initial_position">0.7929</param>
+                    <command_interface name="position" />
+                    <state_interface name="position"/>
+                    <state_interface name="velocity"/>
+                </joint>
+                <joint name="robotiq_85_right_knuckle_joint">
+                    <param name="mimic">robotiq_85_left_knuckle_joint</param>
+                    <param name="multiplier">-1</param>
+                    <command_interface name="position"/>
+                    <state_interface name="position"/>
+                    <state_interface name="velocity"/>
+                </joint>
+                <joint name="robotiq_85_left_inner_knuckle_joint">
+                    <param name="mimic">robotiq_85_left_knuckle_joint</param>
+                    <param name="multiplier">1</param>
+                    <command_interface name="position" />
+                    <state_interface name="position" />
+                    <state_interface name="velocity" />
+                </joint>
+                <joint name="robotiq_85_right_inner_knuckle_joint">
+                    <param name="mimic">robotiq_85_left_knuckle_joint</param>
+                    <param name="multiplier">-1</param>
+                    <command_interface name="position" />
+                    <state_interface name="position" />
+                    <state_interface name="velocity" />
+                </joint>
+                <joint name="robotiq_85_left_finger_tip_joint">
+                    <param name="mimic">robotiq_85_left_knuckle_joint</param>
+                    <param name="multiplier">-1</param>
+                    <command_interface name="position" />
+                    <state_interface name="position" />
+                    <state_interface name="velocity" />
+                </joint>
+                <joint name="robotiq_85_right_finger_tip_joint">
+                    <param name="mimic">robotiq_85_left_knuckle_joint</param>
+                    <param name="multiplier">1</param>
+                    <command_interface name="position" />
+                    <state_interface name="position" />
+                    <state_interface name="velocity" />
+                </joint>
+            </ros2_control>
+            <!--gz plugin for ros2 control -->
+            <xacro:if value="${sim_gz}">
+                <gazebo>
+                    <plugin filename="ign_ros2_control-system" name="ign_ros2_control::IgnitionROS2ControlPlugin">
+                        <parameters>$(find robotiq_driver)/config/robotiq_controllers.yaml</parameters>
+                    </plugin>
+                </gazebo>
+            </xacro:if>
+        </xacro:if>
     </xacro:macro>
 </robot>

File: robotiq_description/urdf/robotiq_gripper.urdf.xacro (robot description, xacro)
@@ -2,9 +2,16 @@
 <robot xmlns:xacro="http://wiki.ros.org/xacro" name="robotiq_gripper">
     <!-- parameters -->
-    <xacro:arg name="use_sim" default="true" />
+    <xacro:arg name="com_port" default="10000" />
+    <xacro:arg name="use_fake_hardware" default="false" />
+    <xacro:arg name="sim_gz" default="true" />
     <!-- Import macros -->
     <xacro:include filename="$(find robotiq_description)/urdf/robotiq_gripper_macro.urdf.xacro" />
     <link name="world" />
-    <xacro:robotiq_gripper parent="world" sim="$(arg use_sim)" prefix="">
+    <xacro:robotiq_gripper
+      parent="world"
+      use_fake_hardware="$(arg use_fake_hardware)"
+      sim_gz="$(arg sim_gz)"
+      com_port="$(arg com_port)"
+      prefix="">
         <origin xyz="0 0 0" rpy="0 0 0" />
     </xacro:robotiq_gripper>

File: robotiq_description/urdf/robotiq_gripper_macro.urdf.xacro (robot description, xacro)
@@ -1,14 +1,26 @@
 <?xml version="1.0"?>
 <robot xmlns:xacro="http://wiki.ros.org/xacro" name="robotiq_gripper">
-    <xacro:macro name="robotiq_gripper" params="parent *origin sim:=false prefix">
+    <!--include macro for ros2_control-->
+    <xacro:include filename="$(find robotiq_description)/urdf/robotiq_gripper.ros2_control.xacro" />
+    <xacro:macro name="robotiq_gripper" params="parent *origin prefix com_port:=10000 use_fake_hardware:=false sim_gz:=true" >
         <link name="${prefix}robotiq_85_base_link">
             <visual>
                 <geometry>
-                    <mesh filename="package://robotiq_description/meshes/visual/robotiq_base.dae" />
-                </geometry>
-            </visual>
-            <collision>
-                <geometry>
-                    <mesh filename="package://robotiq_description/meshes/collision/robotiq_base.stl" />
+                    <xacro:if value="${sim_gz}">
+                        <mesh filename="file://$(find robotiq_description)/meshes/visual/robotiq_base.dae" />
+                    </xacro:if>
+                    <xacro:unless value="${sim_gz}">
+                        <mesh filename="package://robotiq_description/meshes/visual/robotiq_base.dae" />
+                    </xacro:unless>
+                </geometry>
+            </visual>
+            <collision>
+                <geometry>
+                    <xacro:if value="${sim_gz}">
+                        <mesh filename="file://$(find robotiq_description)/meshes/collision/robotiq_base.stl" />
+                    </xacro:if>
+                    <xacro:unless value="${sim_gz}">
+                        <mesh filename="package://robotiq_description/meshes/collision/robotiq_base.stl" />
+                    </xacro:unless>
                 </geometry>
             </collision>
@@ -22,10 +34,20 @@
             <visual>
                 <geometry>
-                    <mesh filename="package://robotiq_description/meshes/visual/left_knuckle.dae" />
-                </geometry>
-            </visual>
-            <collision>
-                <geometry>
-                    <mesh filename="package://robotiq_description/meshes/collision/left_knuckle.stl" />
+                    <xacro:if value="${sim_gz}">
+                        <mesh filename="file://$(find robotiq_description)/meshes/visual/left_knuckle.dae" />
+                    </xacro:if>
+                    <xacro:unless value="${sim_gz}">
+                        <mesh filename="package://robotiq_description/meshes/visual/left_knuckle.dae" />
+                    </xacro:unless>
+                </geometry>
+            </visual>
+            <collision>
+                <geometry>
+                    <xacro:if value="${sim_gz}">
+                        <mesh filename="file://$(find robotiq_description)/meshes/collision/left_knuckle.stl" />
+                    </xacro:if>
+                    <xacro:unless value="${sim_gz}">
+                        <mesh filename="package://robotiq_description/meshes/collision/left_knuckle.stl" />
+                    </xacro:unless>
                 </geometry>
             </collision>
@@ -39,10 +61,20 @@
             <visual>
                 <geometry>
-                    <mesh filename="package://robotiq_description/meshes/visual/right_knuckle.dae" />
-                </geometry>
-            </visual>
-            <collision>
-                <geometry>
-                    <mesh filename="package://robotiq_description/meshes/collision/right_knuckle.stl" />
+                    <xacro:if value="${sim_gz}">
+                        <mesh filename="file://$(find robotiq_description)/meshes/visual/right_knuckle.dae" />
+                    </xacro:if>
+                    <xacro:unless value="${sim_gz}">
+                        <mesh filename="package://robotiq_description/meshes/visual/right_knuckle.dae" />
+                    </xacro:unless>
+                </geometry>
+            </visual>
+            <collision>
+                <geometry>
+                    <xacro:if value="${sim_gz}">
+                        <mesh filename="file://$(find robotiq_description)/meshes/collision/right_knuckle.stl" />
+                    </xacro:if>
+                    <xacro:unless value="${sim_gz}">
+                        <mesh filename="package://robotiq_description/meshes/collision/right_knuckle.stl" />
+                    </xacro:unless>
                 </geometry>
             </collision>
@@ -56,10 +88,20 @@
             <visual>
                 <geometry>
-                    <mesh filename="package://robotiq_description/meshes/visual/left_finger.dae" />
-                </geometry>
-            </visual>
-            <collision>
-                <geometry>
-                    <mesh filename="package://robotiq_description/meshes/collision/left_finger.stl" />
+                    <xacro:if value="${sim_gz}">
+                        <mesh filename="file://$(find robotiq_description)/meshes/visual/left_finger.dae" />
+                    </xacro:if>
+                    <xacro:unless value="${sim_gz}">
+                        <mesh filename="package://robotiq_description/meshes/visual/left_finger.dae" />
+                    </xacro:unless>
+                </geometry>
+            </visual>
+            <collision>
+                <geometry>
+                    <xacro:if value="${sim_gz}">
+                        <mesh filename="file://$(find robotiq_description)/meshes/collision/left_finger.stl" />
+                    </xacro:if>
+                    <xacro:unless value="${sim_gz}">
+                        <mesh filename="package://robotiq_description/meshes/collision/left_finger.stl" />
+                    </xacro:unless>
                 </geometry>
             </collision>
@@ -73,10 +115,20 @@
             <visual>
                 <geometry>
-                    <mesh filename="package://robotiq_description/meshes/visual/right_finger.dae" />
-                </geometry>
-            </visual>
-            <collision>
-                <geometry>
-                    <mesh filename="package://robotiq_description/meshes/collision/right_finger.stl" />
+                    <xacro:if value="${sim_gz}">
+                        <mesh filename="file://$(find robotiq_description)/meshes/visual/right_finger.dae" />
+                    </xacro:if>
+                    <xacro:unless value="${sim_gz}">
+                        <mesh filename="package://robotiq_description/meshes/visual/right_finger.dae" />
+                    </xacro:unless>
+                </geometry>
+            </visual>
+            <collision>
+                <geometry>
+                    <xacro:if value="${sim_gz}">
+                        <mesh filename="file://$(find robotiq_description)/meshes/collision/right_finger.stl" />
+                    </xacro:if>
+                    <xacro:unless value="${sim_gz}">
+                        <mesh filename="package://robotiq_description/meshes/collision/right_finger.stl" />
+                    </xacro:unless>
                 </geometry>
             </collision>
@@ -90,10 +142,20 @@
             <visual>
                 <geometry>
-                    <mesh filename="package://robotiq_description/meshes/visual/left_inner_knuckle.dae" />
-                </geometry>
-            </visual>
-            <collision>
-                <geometry>
-                    <mesh filename="package://robotiq_description/meshes/collision/left_inner_knuckle.stl" />
+                    <xacro:if value="${sim_gz}">
+                        <mesh filename="file://$(find robotiq_description)/meshes/visual/left_inner_knuckle.dae" />
+                    </xacro:if>
+                    <xacro:unless value="${sim_gz}">
+                        <mesh filename="package://robotiq_description/meshes/visual/left_inner_knuckle.dae" />
+                    </xacro:unless>
+                </geometry>
+            </visual>
+            <collision>
+                <geometry>
+                    <xacro:if value="${sim_gz}">
+                        <mesh filename="file://$(find robotiq_description)/meshes/collision/left_inner_knuckle.stl" />
+                    </xacro:if>
+                    <xacro:unless value="${sim_gz}">
+                        <mesh filename="package://robotiq_description/meshes/collision/left_inner_knuckle.stl" />
+                    </xacro:unless>
                 </geometry>
             </collision>
@@ -107,10 +169,20 @@
             <visual>
                 <geometry>
-                    <mesh filename="package://robotiq_description/meshes/visual/right_inner_knuckle.dae" />
-                </geometry>
-            </visual>
-            <collision>
-                <geometry>
-                    <mesh filename="package://robotiq_description/meshes/collision/right_inner_knuckle.stl" />
+                    <xacro:if value="${sim_gz}">
+                        <mesh filename="file://$(find robotiq_description)/meshes/visual/right_inner_knuckle.dae" />
+                    </xacro:if>
+                    <xacro:unless value="${sim_gz}">
+                        <mesh filename="package://robotiq_description/meshes/visual/right_inner_knuckle.dae" />
+                    </xacro:unless>
+                </geometry>
+            </visual>
+            <collision>
+                <geometry>
+                    <xacro:if value="${sim_gz}">
+                        <mesh filename="file://$(find robotiq_description)/meshes/collision/right_inner_knuckle.stl" />
+                    </xacro:if>
+                    <xacro:unless value="${sim_gz}">
+                        <mesh filename="package://robotiq_description/meshes/collision/right_inner_knuckle.stl" />
+                    </xacro:unless>
                 </geometry>
             </collision>
@@ -124,10 +196,20 @@
             <visual>
                 <geometry>
-                    <mesh filename="package://robotiq_description/meshes/visual/left_finger_tip.dae" />
-                </geometry>
-            </visual>
-            <collision>
-                <geometry>
-                    <mesh filename="package://robotiq_description/meshes/collision/left_finger_tip.stl" />
+                    <xacro:if value="${sim_gz}">
+                        <mesh filename="file://$(find robotiq_description)/meshes/visual/left_finger_tip.dae" />
+                    </xacro:if>
+                    <xacro:unless value="${sim_gz}">
+                        <mesh filename="package://robotiq_description/meshes/visual/left_finger_tip.dae" />
+                    </xacro:unless>
+                </geometry>
+            </visual>
+            <collision>
+                <geometry>
+                    <xacro:if value="${sim_gz}">
+                        <mesh filename="file://$(find robotiq_description)/meshes/collision/left_finger_tip.stl" />
+                    </xacro:if>
+                    <xacro:unless value="${sim_gz}">
+                        <mesh filename="package://robotiq_description/meshes/collision/left_finger_tip.stl" />
+                    </xacro:unless>
                 </geometry>
             </collision>
@@ -141,10 +223,20 @@
             <visual>
                 <geometry>
-                    <mesh filename="package://robotiq_description/meshes/visual/right_finger_tip.dae" />
-                </geometry>
-            </visual>
-            <collision>
-                <geometry>
-                    <mesh filename="package://robotiq_description/meshes/collision/right_finger_tip.stl" />
+                    <xacro:if value="${sim_gz}">
+                        <mesh filename="file://$(find robotiq_description)/meshes/visual/right_finger_tip.dae" />
+                    </xacro:if>
+                    <xacro:unless value="${sim_gz}">
+                        <mesh filename="package://robotiq_description/meshes/visual/right_finger_tip.dae" />
+                    </xacro:unless>
+                </geometry>
+            </visual>
+            <collision>
+                <geometry>
+                    <xacro:if value="${sim_gz}">
+                        <mesh filename="file://$(find robotiq_description)/meshes/collision/right_finger_tip.stl" />
+                    </xacro:if>
+                    <xacro:unless value="${sim_gz}">
+                        <mesh filename="package://robotiq_description/meshes/collision/right_finger_tip.stl" />
+                    </xacro:unless>
                 </geometry>
             </collision>
@@ -213,4 +305,10 @@
             <mimic joint="${prefix}robotiq_85_left_knuckle_joint" />
         </joint>
+        <!--instance of robotiq ros2 control hardware interface-->
+        <xacro:robotiq_gripper_ros2_control
+          name="${prefix}robotiq_gripper_hardware_interface"
+          use_fake_hardware="${use_fake_hardware}"
+          sim_gz="${sim_gz}"
+          com_port="${com_port}"/>
     </xacro:macro>
 </robot>
