Commit message: Unify URDF and ros2_control xacro

File: robotiq_description/urdf/robotiq_gripper.ros2_control.xacro (robot description, xacro)
@@ -1,19 +1,100 @@
 <?xml version="1.0"?>
 <robot xmlns:xacro="http://www.ros.org/wiki/xacro">
-    <xacro:macro name="robotiq_gripper_ros2_control" params="name com_port">
-        <ros2_control name="${name}" type="actuator">
+    <xacro:macro name="robotiq_gripper_ros2_control" params="
+        name
+        prefix
+        sim_ignition:=false
+        sim_isaac:=false
+        use_fake_hardware:=false
+        fake_sensor_commands:=false
+        com_port:=/dev/ttyUSB0">
+        <ros2_control name="${name}" type="system">
+            <!-- Plugins -->
             <hardware>
-                <plugin>robotiq_driver/RobotiqGripperHardwareInterface</plugin>
-                <param name="gripper_closed_position">0.7929</param>
-                <param name="COM_port">${com_port}</param>
-                <param name="gripper_speed_multiplier">1.0</param>
-                <param name="gripper_force_multiplier">0.5</param>
+                <xacro:if value="${sim_isaac}">
+                    <plugin>isaac_ros2_control/IsaacSystem</plugin>
+                    <param name="joint_commands_topic">/isaac_joint_commands</param>
+                    <param name="joint_states_topic">/isaac_joint_states</param>
+                </xacro:if>
+                <xacro:if value="${sim_ignition}">
+                    <plugin>ign_ros2_control/IgnitionSystem</plugin>
+                </xacro:if>
+                <xacro:if value="${use_fake_hardware}">
+                    <plugin>mock_components/GenericSystem</plugin>
+                    <param name="fake_sensor_commands">${fake_sensor_commands}</param>
+                    <param name="state_following_offset">0.0</param>
+                </xacro:if>
+                <xacro:unless value="${use_fake_hardware or sim_ignition or sim_isaac}">
+                    <plugin>robotiq_driver/RobotiqGripperHardwareInterface</plugin>
+                    <param name="gripper_closed_position">0.7929</param>
+                    <param name="COM_port">${com_port}</param>
+                    <param name="gripper_speed_multiplier">1.0</param>
+                    <param name="gripper_force_multiplier">0.5</param>
+                </xacro:unless>
             </hardware>
-            <joint name="robotiq_85_left_knuckle_joint">
-                <param name="initial_position">0.7929</param>
+            <!-- Joint interfaces -->
+            <!-- With Ignition or Hardware, they handle mimic joints, so we only need this command interface activated -->
+            <joint name="${prefix}robotiq_85_left_knuckle_joint">
                 <command_interface name="position" />
-                <state_interface name="position" />
-                <state_interface name="velocity" />
+                <state_interface name="position">
+                    <param name="initial_value">0.7929</param>
+                </state_interface>
+                <state_interface name="velocity"/>
             </joint>
+            <!-- When simulating we need to include the rest of the gripper joints -->
+            <xacro:if value="${use_fake_hardware or sim_isaac or sim_ignition}">
+                <joint name="${prefix}robotiq_85_right_knuckle_joint">
+                    <param name="mimic">robotiq_85_left_knuckle_joint</param>
+                    <param name="multiplier">-1</param>
+                    <xacro:unless value="${sim_ignition}">
+                        <command_interface name="position"/>
+                        <state_interface name="position"/>
+                        <state_interface name="velocity"/>
+                    </xacro:unless>
+                </joint>
+                <joint name="${prefix}robotiq_85_left_inner_knuckle_joint">
+                    <param name="mimic">robotiq_85_left_knuckle_joint</param>
+                    <param name="multiplier">1</param>
+                    <xacro:unless value="${sim_ignition}">
+                        <command_interface name="position"/>
+                        <state_interface name="position"/>
+                        <state_interface name="velocity"/>
+                    </xacro:unless>
+                </joint>
+                <joint name="${prefix}robotiq_85_right_inner_knuckle_joint">
+                    <param name="mimic">robotiq_85_left_knuckle_joint</param>
+                    <param name="multiplier">-1</param>
+                    <xacro:unless value="${sim_ignition}">
+                        <command_interface name="position"/>
+                        <state_interface name="position"/>
+                        <state_interface name="velocity"/>
+                    </xacro:unless>
+                </joint>
+                <joint name="${prefix}robotiq_85_left_finger_tip_joint">
+                    <param name="mimic">robotiq_85_left_knuckle_joint</param>
+                    <param name="multiplier">-1</param>
+                    <xacro:unless value="${sim_ignition}">
+                        <command_interface name="position"/>
+                        <state_interface name="position"/>
+                        <state_interface name="velocity"/>
+                    </xacro:unless>
+                </joint>
+                <joint name="${prefix}robotiq_85_right_finger_tip_joint">
+                    <param name="mimic">robotiq_85_left_knuckle_joint</param>
+                    <param name="multiplier">1</param>
+                    <xacro:unless value="${sim_ignition}">
+                        <command_interface name="position"/>
+                        <state_interface name="position"/>
+                        <state_interface name="velocity"/>
+                    </xacro:unless>
+                </joint>
+            </xacro:if>
+            <!-- Only add this with fake hardware mode -->
+            <xacro:unless value="${sim_ignition or sim_isaac}">
+                <gpio name="reactivate_gripper">
+                    <command_interface name="reactivate_gripper_cmd" />
+                    <command_interface name="reactivate_gripper_response" />
+                </gpio>
+            </xacro:unless>
         </ros2_control>
     </xacro:macro>

File: robotiq_description/urdf/robotiq_gripper_macro.urdf.xacro (robot description, xacro)
@@ -1,5 +1,25 @@
 <?xml version="1.0"?>
 <robot xmlns:xacro="http://wiki.ros.org/xacro" name="robotiq_gripper">
-    <xacro:macro name="robotiq_gripper" params="parent *origin sim:=false prefix">
+    <xacro:macro name="robotiq_gripper" params="
+        name
+        prefix
+        parent
+        *origin
+        sim_ignition:=false
+        sim_isaac:=false
+        use_fake_hardware:=false
+        fake_sensor_commands:=false
+        com_port:=/dev/ttyUSB0">
+        <!-- ros2 control include -->
+        <xacro:include filename="$(find robotiq_description)/urdf/robotiq_gripper.ros2_control.xacro" />
+        <!-- ros2 control instance -->
+        <xacro:robotiq_gripper_ros2_control
+            name="${name}" prefix="${prefix}"
+            sim_ignition="${sim_ignition}"
+            sim_isaac="${sim_isaac}"
+            use_fake_hardware="${use_fake_hardware}"
+            fake_sensor_commands="${fake_sensor_commands}"
+            com_port="${com_port}"
+            />
         <link name="${prefix}robotiq_85_base_link">
             <visual>
