Commit message: Add mass properties.

File: robotiq_description/urdf/robotiq_gripper_macro.urdf.xacro (robot description, xacro)
@@ -11,4 +11,9 @@
                 </geometry>
             </visual>
+            <inertial>
+                <origin xyz="0.0 2.274e-05 0.03232288" rpy="0 0 0" />
+                <mass value="6.6320197e-01" />
+                <inertia ixx="5.1617816e-04" iyy="5.8802208e-04" izz="3.9462776e-04" ixy="2.936e-8" ixz="0.0" iyz="-3.2296e-7" />
+            </inertial>
         </link>
         <link name="${prefix}robotiq_85_left_knuckle_link">
@@ -18,4 +23,9 @@
                 </geometry>
             </visual>
+            <inertial>
+                <origin xyz="0.01213197 0.0002 -0.00058647" rpy="0 0 0" />
+                <mass value="1.384773208e-02" />
+                <inertia ixx="3.5232e-7" iyy="2.31944e-6" izz="2.23136e-6" ixy="0.0" ixz="1.1744e-7" iyz="0" />
+            </inertial>
         </link>
         <link name="${prefix}robotiq_85_right_knuckle_link">
@@ -25,4 +35,9 @@
                 </geometry>
             </visual>
+            <inertial>
+                <origin xyz="-0.01213197 0.0002 -0.00058647" rpy="0 0 0" />
+                <mass value="1.384773208e-02" />
+                <inertia ixx="3.5232e-7" iyy="2.31944e-6" izz="2.23136e-6" ixy="0.0" ixz="-1.1744e-7" iyz="0.0" />
+            </inertial>
         </link>
         <link name="${prefix}robotiq_85_left_finger_link">
@@ -32,4 +47,9 @@
                 </geometry>
             </visual>
+            <inertial>
+                <origin xyz="0.00346899 -0.00079447 0.01867121" rpy="0 0 0" />
+                <mass value="4.260376752e-02" />
+                <inertia ixx="1.385792000000000e-05" iyy="1.183208e-05" izz="5.19672e-06" ixy="0.0" ixz="-2.17264e-06" iyz="0.0" />
+            </inertial>
         </link>
         <link name="${prefix}robotiq_85_right_finger_link">
@@ -39,4 +59,9 @@
                 </geometry>
             </visual>
+            <inertial>
+                <origin xyz="-0.00346899 -5.53e-06 0.01867121" rpy="0 0 0" />
+                <mass value="4.260376752000000e-02" />
+                <inertia ixx="1.385792e-05" iyy="1.183208e-05" izz="5.19672e-06" ixy="0.0" ixz="2.17264e-06" iyz="0.0" />
+            </inertial>
         </link>
         <link name="${prefix}robotiq_85_left_inner_knuckle_link">
@@ -46,4 +71,9 @@
                 </geometry>
             </visual>
+            <inertial>
+                <origin xyz="0.01897699 0.00015001 0.02247101" rpy="0 0 0" />
+                <mass value="2.969376448e-02" />
+                <inertia ixx="9.57136e-06" iyy="8.69056e-06" izz="8.19144e-06" ixy="0.0" ixz="-3.93424e-06" iyz="0.0" />
+            </inertial>
         </link>
         <link name="${prefix}robotiq_85_right_inner_knuckle_link">
@@ -53,4 +83,9 @@
                 </geometry>
             </visual>
+            <inertial>
+                <origin xyz="-0.01926824 5.001e-05 0.02222178" rpy="0 0 0" />
+                <mass value="2.969376448e-02" />
+                <inertia ixx="9.42456e-06" iyy="8.69056e-06" izz="8.33824e-06" ixy="0.0" ixz="3.9636e-06" iyz="0.0" />
+            </inertial>
         </link>
         <link name="${prefix}robotiq_85_left_finger_tip_link">
@@ -60,4 +95,9 @@
                 </geometry>
             </visual>
+            <inertial>
+                <origin xyz="-0.01456706 -0.0008 0.01649701" rpy="0 0 0" />
+                <mass value="4.268588744e-02" />
+                <inertia ixx="1.048152e-05" iyy="1.197888e-05" izz="4.22784e-06" ixy="0.0" ixz="3.5232e-6" iyz="0.0" />
+            </inertial>
         </link>
         <link name="${prefix}robotiq_85_right_finger_tip_link">
@@ -67,4 +107,9 @@
                 </geometry>
             </visual>
+            <inertial>
+                <origin xyz="0.01456706 5e-05 0.01649701" rpy="0 0 0" />
+                <mass value="4.268588744e-02" />
+                <inertia ixx="1.048152e-05" iyy="1.197888e-05" izz="4.22784e-06" ixy="0.0" ixz="-3.5232e-06" iyz="0.0" />
+            </inertial>
         </link>
         <joint name="${prefix}robotiq_85_base_joint" type="fixed">

Commit message: Add mimic joints.

File: robotiq_description/urdf/robotiq_gripper_macro.urdf.xacro (robot description, xacro)
@@ -128,4 +128,5 @@
             <origin xyz="-0.03060114 0.0 0.05490452" rpy="0 0 0" />
             <limit lower="-0.8" upper="0.0" velocity="0.5" effort="50" />
+            <mimic joint="${prefix}robotiq_85_left_knuckle_joint" multiplier="-1" />
         </joint>
         <joint name="${prefix}robotiq_85_left_finger_joint" type="fixed">
@@ -144,4 +145,5 @@
             <axis xyz="0 1 0" />
             <origin xyz="0.0127 0.0 0.06142" rpy="0 0 0" />
+            <mimic joint="robotiq_85_left_knuckle_joint" />
         </joint>
         <joint name="${prefix}robotiq_85_right_inner_knuckle_joint" type="continuous">
@@ -150,16 +152,19 @@
             <axis xyz="0 1 0" />
             <origin xyz="-0.0127 0.0 0.06142" rpy="0 0 0" />
+            <mimic joint="robotiq_85_left_knuckle_joint" multiplier="-1" />
         </joint>
         <joint name="${prefix}robotiq_85_left_finger_tip_joint" type="continuous">
             <parent link="${prefix}robotiq_85_left_finger_link" />
             <child link="${prefix}robotiq_85_left_finger_tip_link" />
-            <axis xyz="1 0 0" />
+            <axis xyz="0 1 0" />
             <origin xyz="0.00563134 0.0 0.04718515" rpy="0 0 0" />
+            <mimic joint="robotiq_85_left_knuckle_joint" multiplier="-1" />
         </joint>
         <joint name="${prefix}robotiq_85_right_finger_tip_joint" type="continuous">
             <parent link="${prefix}robotiq_85_right_finger_link" />
             <child link="${prefix}robotiq_85_right_finger_tip_link" />
-            <axis xyz="1 0 0" />
+            <axis xyz="0 1 0" />
             <origin xyz="-0.00563134 0.0 0.04718515" rpy="0 0 0" />
+            <mimic joint="robotiq_85_left_knuckle_joint" />
         </joint>
         <xacro:unless value="$(arg use_sim)">

Commit message: Adjust joint limits.

File: robotiq_description/urdf/robotiq_gripper_macro.urdf.xacro (robot description, xacro)
@@ -120,5 +120,5 @@
             <axis xyz="0 1 0" />
             <origin xyz="0.03060114 0.0 0.05490452" rpy="0 0 0" />
-            <limit lower="0.0" upper="0.8" velocity="0.5" effort="50" />
+            <limit lower="-0.8" upper="0.0" velocity="0.5" effort="50" />
         </joint>
         <joint name="${prefix}robotiq_85_right_knuckle_joint" type="revolute">
@@ -127,5 +127,5 @@
             <axis xyz="0 1 0" />
             <origin xyz="-0.03060114 0.0 0.05490452" rpy="0 0 0" />
-            <limit lower="-0.8" upper="0.0" velocity="0.5" effort="50" />
+            <limit lower="0.0" upper="0.8" velocity="0.5" effort="50" />
             <mimic joint="${prefix}robotiq_85_left_knuckle_joint" multiplier="-1" />
         </joint>

File: robotiq_description/urdf/robotiq_sim_gripper.ros2_control.xacro (robot description, xacro)
@@ -6,5 +6,5 @@
                 <plugin>fake_components/GenericSystem</plugin>
             </hardware>
-            <joint name="finger_joint">
+            <joint name="robotiq_85_left_knuckle_joint">
                 <param name="initial_position">0.7929</param>
                 <command_interface name="position" />

Commit message: Invert joint axes.

File: robotiq_description/urdf/robotiq_gripper_macro.urdf.xacro (robot description, xacro)
@@ -118,14 +118,14 @@
             <parent link="${prefix}robotiq_85_base_link" />
             <child link="${prefix}robotiq_85_left_knuckle_link" />
-            <axis xyz="0 1 0" />
+            <axis xyz="0 -1 0" />
             <origin xyz="0.03060114 0.0 0.05490452" rpy="0 0 0" />
-            <limit lower="-0.8" upper="0.0" velocity="0.5" effort="50" />
+            <limit lower="0.0" upper="0.8" velocity="0.5" effort="50" />
         </joint>
         <joint name="${prefix}robotiq_85_right_knuckle_joint" type="revolute">
             <parent link="${prefix}robotiq_85_base_link" />
             <child link="${prefix}robotiq_85_right_knuckle_link" />
-            <axis xyz="0 1 0" />
+            <axis xyz="0 -1 0" />
             <origin xyz="-0.03060114 0.0 0.05490452" rpy="0 0 0" />
-            <limit lower="0.0" upper="0.8" velocity="0.5" effort="50" />
+            <limit lower="-0.8" upper="0.0" velocity="0.5" effort="50" />
             <mimic joint="${prefix}robotiq_85_left_knuckle_joint" multiplier="-1" />
         </joint>
@@ -143,5 +143,5 @@
             <parent link="${prefix}robotiq_85_base_link" />
             <child link="${prefix}robotiq_85_left_inner_knuckle_link" />
-            <axis xyz="0 1 0" />
+            <axis xyz="0 -1 0" />
             <origin xyz="0.0127 0.0 0.06142" rpy="0 0 0" />
             <mimic joint="robotiq_85_left_knuckle_joint" />
@@ -150,5 +150,5 @@
             <parent link="${prefix}robotiq_85_base_link" />
             <child link="${prefix}robotiq_85_right_inner_knuckle_link" />
-            <axis xyz="0 1 0" />
+            <axis xyz="0 -1 0" />
             <origin xyz="-0.0127 0.0 0.06142" rpy="0 0 0" />
             <mimic joint="robotiq_85_left_knuckle_joint" multiplier="-1" />
@@ -157,5 +157,5 @@
             <parent link="${prefix}robotiq_85_left_finger_link" />
             <child link="${prefix}robotiq_85_left_finger_tip_link" />
-            <axis xyz="0 1 0" />
+            <axis xyz="0 -1 0" />
             <origin xyz="0.00563134 0.0 0.04718515" rpy="0 0 0" />
             <mimic joint="robotiq_85_left_knuckle_joint" multiplier="-1" />
@@ -164,5 +164,5 @@
             <parent link="${prefix}robotiq_85_right_finger_link" />
             <child link="${prefix}robotiq_85_right_finger_tip_link" />
-            <axis xyz="0 1 0" />
+            <axis xyz="0 -1 0" />
             <origin xyz="-0.00563134 0.0 0.04718515" rpy="0 0 0" />
             <mimic joint="robotiq_85_left_knuckle_joint" />

Commit message: Add visual meshes and simplified collision meshes.

File: robotiq_description/urdf/robotiq_gripper_macro.urdf.xacro (robot description, xacro)
@@ -5,7 +5,12 @@
             <visual>
                 <geometry>
+                    <mesh filename="package://robotiq_description/meshes/visual/robotiq_base.dae" />
+                </geometry>
+            </visual>
+            <collision>
+                <geometry>
                     <mesh filename="package://robotiq_description/meshes/collision/robotiq_base.stl" />
                 </geometry>
-            </visual>
+            </collision>
             <inertial>
                 <origin xyz="0.0 2.274e-05 0.03232288" rpy="0 0 0" />
@@ -17,7 +22,12 @@
             <visual>
                 <geometry>
+                    <mesh filename="package://robotiq_description/meshes/visual/left_knuckle.dae" />
+                </geometry>
+            </visual>
+            <collision>
+                <geometry>
                     <mesh filename="package://robotiq_description/meshes/collision/left_knuckle.stl" />
                 </geometry>
-            </visual>
+            </collision>
             <inertial>
                 <origin xyz="0.01213197 0.0002 -0.00058647" rpy="0 0 0" />
@@ -29,7 +39,12 @@
             <visual>
                 <geometry>
+                    <mesh filename="package://robotiq_description/meshes/visual/right_knuckle.dae" />
+                </geometry>
+            </visual>
+            <collision>
+                <geometry>
                     <mesh filename="package://robotiq_description/meshes/collision/right_knuckle.stl" />
                 </geometry>
-            </visual>
+            </collision>
             <inertial>
                 <origin xyz="-0.01213197 0.0002 -0.00058647" rpy="0 0 0" />
@@ -41,7 +56,12 @@
             <visual>
                 <geometry>
+                    <mesh filename="package://robotiq_description/meshes/visual/left_finger.dae" />
+                </geometry>
+            </visual>
+            <collision>
+                <geometry>
                     <mesh filename="package://robotiq_description/meshes/collision/left_finger.stl" />
                 </geometry>
-            </visual>
+            </collision>
             <inertial>
                 <origin xyz="0.00346899 -0.00079447 0.01867121" rpy="0 0 0" />
@@ -53,7 +73,12 @@
             <visual>
                 <geometry>
+                    <mesh filename="package://robotiq_description/meshes/visual/right_finger.dae" />
+                </geometry>
+            </visual>
+            <collision>
+                <geometry>
                     <mesh filename="package://robotiq_description/meshes/collision/right_finger.stl" />
                 </geometry>
-            </visual>
+            </collision>
             <inertial>
                 <origin xyz="-0.00346899 -5.53e-06 0.01867121" rpy="0 0 0" />
@@ -65,7 +90,12 @@
             <visual>
                 <geometry>
+                    <mesh filename="package://robotiq_description/meshes/visual/left_inner_knuckle.dae" />
+                </geometry>
+            </visual>
+            <collision>
+                <geometry>
                     <mesh filename="package://robotiq_description/meshes/collision/left_inner_knuckle.stl" />
                 </geometry>
-            </visual>
+            </collision>
             <inertial>
                 <origin xyz="0.01897699 0.00015001 0.02247101" rpy="0 0 0" />
@@ -77,7 +107,12 @@
             <visual>
                 <geometry>
+                    <mesh filename="package://robotiq_description/meshes/visual/right_inner_knuckle.dae" />
+                </geometry>
+            </visual>
+            <collision>
+                <geometry>
                     <mesh filename="package://robotiq_description/meshes/collision/right_inner_knuckle.stl" />
                 </geometry>
-            </visual>
+            </collision>
             <inertial>
                 <origin xyz="-0.01926824 5.001e-05 0.02222178" rpy="0 0 0" />
@@ -89,7 +124,12 @@
             <visual>
                 <geometry>
+                    <mesh filename="package://robotiq_description/meshes/visual/left_finger_tip.dae" />
+                </geometry>
+            </visual>
+            <collision>
+                <geometry>
                     <mesh filename="package://robotiq_description/meshes/collision/left_finger_tip.stl" />
                 </geometry>
-            </visual>
+            </collision>
             <inertial>
                 <origin xyz="-0.01456706 -0.0008 0.01649701" rpy="0 0 0" />
@@ -101,7 +141,12 @@
             <visual>
                 <geometry>
+                    <mesh filename="package://robotiq_description/meshes/visual/right_finger_tip.dae" />
+                </geometry>
+            </visual>
+            <collision>
+                <geometry>
                     <mesh filename="package://robotiq_description/meshes/collision/right_finger_tip.stl" />
                 </geometry>
-            </visual>
+            </collision>
             <inertial>
                 <origin xyz="0.01456706 5e-05 0.01649701" rpy="0 0 0" />

Commit message: Fix missing prefix for mimic joints.

File: robotiq_description/urdf/robotiq_gripper_macro.urdf.xacro (robot description, xacro)
@@ -190,5 +190,5 @@
             <axis xyz="0 -1 0" />
             <origin xyz="0.0127 0.0 0.06142" rpy="0 0 0" />
-            <mimic joint="robotiq_85_left_knuckle_joint" />
+            <mimic joint="${prefix}robotiq_85_left_knuckle_joint" />
         </joint>
         <joint name="${prefix}robotiq_85_right_inner_knuckle_joint" type="continuous">
@@ -197,5 +197,5 @@
             <axis xyz="0 -1 0" />
             <origin xyz="-0.0127 0.0 0.06142" rpy="0 0 0" />
-            <mimic joint="robotiq_85_left_knuckle_joint" multiplier="-1" />
+            <mimic joint="${prefix}robotiq_85_left_knuckle_joint" multiplier="-1" />
         </joint>
         <joint name="${prefix}robotiq_85_left_finger_tip_joint" type="continuous">
@@ -204,5 +204,5 @@
             <axis xyz="0 -1 0" />
             <origin xyz="0.00563134 0.0 0.04718515" rpy="0 0 0" />
-            <mimic joint="robotiq_85_left_knuckle_joint" multiplier="-1" />
+            <mimic joint="${prefix}robotiq_85_left_knuckle_joint" multiplier="-1" />
         </joint>
         <joint name="${prefix}robotiq_85_right_finger_tip_joint" type="continuous">
@@ -211,5 +211,5 @@
             <axis xyz="0 -1 0" />
             <origin xyz="-0.00563134 0.0 0.04718515" rpy="0 0 0" />
-            <mimic joint="robotiq_85_left_knuckle_joint" />
+            <mimic joint="${prefix}robotiq_85_left_knuckle_joint" />
         </joint>
     </xacro:macro>
