Commit message: Add ros2_control switch and enable mesh loadingin Gazebo

File: robotiq_description/urdf/robotiq_gripper_macro.urdf.xacro (robot description, xacro)
@@ -10,25 +10,27 @@
         use_fake_hardware:=false
         fake_sensor_commands:=false
+        include_ros2_control:=true
         com_port:=/dev/ttyUSB0">
         <!-- ros2 control include -->
         <xacro:include filename="$(find robotiq_description)/urdf/robotiq_gripper.ros2_control.xacro" />
-        <!-- ros2 control instance -->
-        <xacro:robotiq_gripper_ros2_control
-            name="${name}" prefix="${prefix}"
-            sim_ignition="${sim_ignition}"
-            sim_isaac="${sim_isaac}"
-            use_fake_hardware="${use_fake_hardware}"
-            fake_sensor_commands="${fake_sensor_commands}"
-            com_port="${com_port}"
-            />
+        <!-- if we are simulating or directly communicating with the gripper we need a ros2 control instance -->
+        <xacro:if value="${include_ros2_control}">
+            <xacro:robotiq_gripper_ros2_control
+                name="${name}" prefix="${prefix}"
+                sim_ignition="${sim_ignition}"
+                sim_isaac="${sim_isaac}"
+                use_fake_hardware="${use_fake_hardware}"
+                fake_sensor_commands="${fake_sensor_commands}"
+                com_port="${com_port}"/>
+        </xacro:if>
         <link name="${prefix}robotiq_85_base_link">
             <visual>
                 <geometry>
-                    <mesh filename="package://robotiq_description/meshes/visual/robotiq_base.dae" />
-                </geometry>
-            </visual>
-            <collision>
-                <geometry>
-                    <mesh filename="package://robotiq_description/meshes/collision/robotiq_base.stl" />
+                    <mesh filename="$(find robotiq_description)/meshes/visual/robotiq_base.dae" />
+                </geometry>
+            </visual>
+            <collision>
+                <geometry>
+                    <mesh filename="$(find robotiq_description)/meshes/collision/robotiq_base.stl" />
                 </geometry>
             </collision>
@@ -42,10 +44,10 @@
             <visual>
                 <geometry>
-                    <mesh filename="package://robotiq_description/meshes/visual/left_knuckle.dae" />
-                </geometry>
-            </visual>
-            <collision>
-                <geometry>
-                    <mesh filename="package://robotiq_description/meshes/collision/left_knuckle.stl" />
+                    <mesh filename="$(find robotiq_description)/meshes/visual/left_knuckle.dae" />
+                </geometry>
+            </visual>
+            <collision>
+                <geometry>
+                    <mesh filename="$(find robotiq_description)/meshes/collision/left_knuckle.stl" />
                 </geometry>
             </collision>
@@ -59,10 +61,10 @@
             <visual>
                 <geometry>
-                    <mesh filename="package://robotiq_description/meshes/visual/right_knuckle.dae" />
-                </geometry>
-            </visual>
-            <collision>
-                <geometry>
-                    <mesh filename="package://robotiq_description/meshes/collision/right_knuckle.stl" />
+                    <mesh filename="$(find robotiq_description)/meshes/visual/right_knuckle.dae" />
+                </geometry>
+            </visual>
+            <collision>
+                <geometry>
+                    <mesh filename="$(find robotiq_description)/meshes/collision/right_knuckle.stl" />
                 </geometry>
             </collision>
@@ -76,10 +78,10 @@
             <visual>
                 <geometry>
-                    <mesh filename="package://robotiq_description/meshes/visual/left_finger.dae" />
-                </geometry>
-            </visual>
-            <collision>
-                <geometry>
-                    <mesh filename="package://robotiq_description/meshes/collision/left_finger.stl" />
+                    <mesh filename="$(find robotiq_description)/meshes/visual/left_finger.dae" />
+                </geometry>
+            </visual>
+            <collision>
+                <geometry>
+                    <mesh filename="$(find robotiq_description)/meshes/collision/left_finger.stl" />
                 </geometry>
             </collision>
@@ -93,10 +95,10 @@
             <visual>
                 <geometry>
-                    <mesh filename="package://robotiq_description/meshes/visual/right_finger.dae" />
-                </geometry>
-            </visual>
-            <collision>
-                <geometry>
-                    <mesh filename="package://robotiq_description/meshes/collision/right_finger.stl" />
+                    <mesh filename="$(find robotiq_description)/meshes/visual/right_finger.dae" />
+                </geometry>
+            </visual>
+            <collision>
+                <geometry>
+                    <mesh filename="$(find robotiq_description)/meshes/collision/right_finger.stl" />
                 </geometry>
             </collision>
@@ -110,10 +112,10 @@
             <visual>
                 <geometry>
-                    <mesh filename="package://robotiq_description/meshes/visual/left_inner_knuckle.dae" />
-                </geometry>
-            </visual>
-            <collision>
-                <geometry>
-                    <mesh filename="package://robotiq_description/meshes/collision/left_inner_knuckle.stl" />
+                    <mesh filename="$(find robotiq_description)/meshes/visual/left_inner_knuckle.dae" />
+                </geometry>
+            </visual>
+            <collision>
+                <geometry>
+                    <mesh filename="$(find robotiq_description)/meshes/collision/left_inner_knuckle.stl" />
                 </geometry>
             </collision>
@@ -127,10 +129,10 @@
             <visual>
                 <geometry>
-                    <mesh filename="package://robotiq_description/meshes/visual/right_inner_knuckle.dae" />
-                </geometry>
-            </visual>
-            <collision>
-                <geometry>
-                    <mesh filename="package://robotiq_description/meshes/collision/right_inner_knuckle.stl" />
+                    <mesh filename="$(find robotiq_description)/meshes/visual/right_inner_knuckle.dae" />
+                </geometry>
+            </visual>
+            <collision>
+                <geometry>
+                    <mesh filename="$(find robotiq_description)/meshes/collision/right_inner_knuckle.stl" />
                 </geometry>
             </collision>
@@ -144,10 +146,10 @@
             <visual>
                 <geometry>
-                    <mesh filename="package://robotiq_description/meshes/visual/left_finger_tip.dae" />
-                </geometry>
-            </visual>
-            <collision>
-                <geometry>
-                    <mesh filename="package://robotiq_description/meshes/collision/left_finger_tip.stl" />
+                    <mesh filename="$(find robotiq_description)/meshes/visual/left_finger_tip.dae" />
+                </geometry>
+            </visual>
+            <collision>
+                <geometry>
+                    <mesh filename="$(find robotiq_description)/meshes/collision/left_finger_tip.stl" />
                 </geometry>
                 <surface>
@@ -179,10 +181,10 @@
             <visual>
                 <geometry>
-                    <mesh filename="package://robotiq_description/meshes/visual/right_finger_tip.dae" />
-                </geometry>
-            </visual>
-            <collision>
-                <geometry>
-                    <mesh filename="package://robotiq_description/meshes/collision/right_finger_tip.stl" />
+                    <mesh filename="$(find robotiq_description)/meshes/visual/right_finger_tip.dae" />
+                </geometry>
+            </visual>
+            <collision>
+                <geometry>
+                    <mesh filename="$(find robotiq_description)/meshes/collision/right_finger_tip.stl" />
                 </geometry>
                 <surface>

Commit message: add missing file:// tag

File: robotiq_description/urdf/robotiq_gripper_macro.urdf.xacro (robot description, xacro)
@@ -27,10 +27,10 @@
             <visual>
                 <geometry>
-                    <mesh filename="$(find robotiq_description)/meshes/visual/robotiq_base.dae" />
-                </geometry>
-            </visual>
-            <collision>
-                <geometry>
-                    <mesh filename="$(find robotiq_description)/meshes/collision/robotiq_base.stl" />
+                    <mesh filename="file://$(find robotiq_description)/meshes/visual/robotiq_base.dae" />
+                </geometry>
+            </visual>
+            <collision>
+                <geometry>
+                    <mesh filename="file://$(find robotiq_description)/meshes/collision/robotiq_base.stl" />
                 </geometry>
             </collision>
@@ -44,10 +44,10 @@
             <visual>
                 <geometry>
-                    <mesh filename="$(find robotiq_description)/meshes/visual/left_knuckle.dae" />
-                </geometry>
-            </visual>
-            <collision>
-                <geometry>
-                    <mesh filename="$(find robotiq_description)/meshes/collision/left_knuckle.stl" />
+                    <mesh filename="file://$(find robotiq_description)/meshes/visual/left_knuckle.dae" />
+                </geometry>
+            </visual>
+            <collision>
+                <geometry>
+                    <mesh filename="file://$(find robotiq_description)/meshes/collision/left_knuckle.stl" />
                 </geometry>
             </collision>
@@ -61,10 +61,10 @@
             <visual>
                 <geometry>
-                    <mesh filename="$(find robotiq_description)/meshes/visual/right_knuckle.dae" />
-                </geometry>
-            </visual>
-            <collision>
-                <geometry>
-                    <mesh filename="$(find robotiq_description)/meshes/collision/right_knuckle.stl" />
+                    <mesh filename="file://$(find robotiq_description)/meshes/visual/right_knuckle.dae" />
+                </geometry>
+            </visual>
+            <collision>
+                <geometry>
+                    <mesh filename="file://$(find robotiq_description)/meshes/collision/right_knuckle.stl" />
                 </geometry>
             </collision>
@@ -78,10 +78,10 @@
             <visual>
                 <geometry>
-                    <mesh filename="$(find robotiq_description)/meshes/visual/left_finger.dae" />
-                </geometry>
-            </visual>
-            <collision>
-                <geometry>
-                    <mesh filename="$(find robotiq_description)/meshes/collision/left_finger.stl" />
+                    <mesh filename="file://$(find robotiq_description)/meshes/visual/left_finger.dae" />
+                </geometry>
+            </visual>
+            <collision>
+                <geometry>
+                    <mesh filename="file://$(find robotiq_description)/meshes/collision/left_finger.stl" />
                 </geometry>
             </collision>
@@ -95,10 +95,10 @@
             <visual>
                 <geometry>
-                    <mesh filename="$(find robotiq_description)/meshes/visual/right_finger.dae" />
-                </geometry>
-            </visual>
-            <collision>
-                <geometry>
-                    <mesh filename="$(find robotiq_description)/meshes/collision/right_finger.stl" />
+                    <mesh filename="file://$(find robotiq_description)/meshes/visual/right_finger.dae" />
+                </geometry>
+            </visual>
+            <collision>
+                <geometry>
+                    <mesh filename="file://$(find robotiq_description)/meshes/collision/right_finger.stl" />
                 </geometry>
             </collision>
@@ -112,10 +112,10 @@
             <visual>
                 <geometry>
-                    <mesh filename="$(find robotiq_description)/meshes/visual/left_inner_knuckle.dae" />
-                </geometry>
-            </visual>
-            <collision>
-                <geometry>
-                    <mesh filename="$(find robotiq_description)/meshes/collision/left_inner_knuckle.stl" />
+                    <mesh filename="file://$(find robotiq_description)/meshes/visual/left_inner_knuckle.dae" />
+                </geometry>
+            </visual>
+            <collision>
+                <geometry>
+                    <mesh filename="file://$(find robotiq_description)/meshes/collision/left_inner_knuckle.stl" />
                 </geometry>
             </collision>
@@ -129,10 +129,10 @@
             <visual>
                 <geometry>
-                    <mesh filename="$(find robotiq_description)/meshes/visual/right_inner_knuckle.dae" />
-                </geometry>
-            </visual>
-            <collision>
-                <geometry>
-                    <mesh filename="$(find robotiq_description)/meshes/collision/right_inner_knuckle.stl" />
+                    <mesh filename="file://$(find robotiq_description)/meshes/visual/right_inner_knuckle.dae" />
+                </geometry>
+            </visual>
+            <collision>
+                <geometry>
+                    <mesh filename="file://$(find robotiq_description)/meshes/collision/right_inner_knuckle.stl" />
                 </geometry>
             </collision>
@@ -146,10 +146,10 @@
             <visual>
                 <geometry>
-                    <mesh filename="$(find robotiq_description)/meshes/visual/left_finger_tip.dae" />
-                </geometry>
-            </visual>
-            <collision>
-                <geometry>
-                    <mesh filename="$(find robotiq_description)/meshes/collision/left_finger_tip.stl" />
+                    <mesh filename="file://$(find robotiq_description)/meshes/visual/left_finger_tip.dae" />
+                </geometry>
+            </visual>
+            <collision>
+                <geometry>
+                    <mesh filename="file://$(find robotiq_description)/meshes/collision/left_finger_tip.stl" />
                 </geometry>
                 <surface>
@@ -181,10 +181,10 @@
             <visual>
                 <geometry>
-                    <mesh filename="$(find robotiq_description)/meshes/visual/right_finger_tip.dae" />
-                </geometry>
-            </visual>
-            <collision>
-                <geometry>
-                    <mesh filename="$(find robotiq_description)/meshes/collision/right_finger_tip.stl" />
+                    <mesh filename="file://$(find robotiq_description)/meshes/visual/right_finger_tip.dae" />
+                </geometry>
+            </visual>
+            <collision>
+                <geometry>
+                    <mesh filename="file://$(find robotiq_description)/meshes/collision/right_finger_tip.stl" />
                 </geometry>
                 <surface>
