Commit message: Replace find with package

File: robotiq_description/urdf/robotiq_2f_85_gripper.urdf.xacro (robot description, xacro)
@@ -4,5 +4,5 @@
     <xacro:arg name="use_fake_hardware" default="true" />
     <!-- Import macros -->
-    <xacro:include filename="$(find robotiq_description)/urdf/robotiq_2f_85_macro.urdf.xacro" />
+    <xacro:include filename="package://robotiq_description/urdf/robotiq_2f_85_macro.urdf.xacro" />
     <link name="world" />
     <xacro:robotiq_gripper name="RobotiqGripperHardwareInterface" prefix="" parent="world" use_fake_hardware="$(arg use_fake_hardware)">

File: robotiq_description/urdf/robotiq_2f_85_macro.urdf.xacro (robot description, xacro)
@@ -13,5 +13,5 @@
         com_port:=/dev/ttyUSB0">
         <!-- ros2 control include -->
-        <xacro:include filename="$(find robotiq_description)/urdf/robotiq_gripper.ros2_control.xacro" />
+        <xacro:include filename="package://robotiq_description/urdf/robotiq_gripper.ros2_control.xacro" />
         <!-- if we are simulating or directly communicating with the gripper we need a ros2 control instance -->
         <xacro:if value="${include_ros2_control}">
@@ -27,10 +27,10 @@
             <visual>
                 <geometry>
-                    <mesh filename="file://$(find robotiq_description)/meshes/visual/robotiq_base.dae" />
-                </geometry>
-            </visual>
-            <collision>
-                <geometry>
-                    <mesh filename="file://$(find robotiq_description)/meshes/collision/robotiq_base.stl" />
+                    <mesh filename="package://robotiq_description/meshes/visual/robotiq_base.dae" />
+                </geometry>
+            </visual>
+            <collision>
+                <geometry>
+                    <mesh filename="package://robotiq_description/meshes/collision/robotiq_base.stl" />
                 </geometry>
             </collision>
@@ -44,10 +44,10 @@
             <visual>
                 <geometry>
-                    <mesh filename="file://$(find robotiq_description)/meshes/visual/left_knuckle.dae" />
-                </geometry>
-            </visual>
-            <collision>
-                <geometry>
-                    <mesh filename="file://$(find robotiq_description)/meshes/collision/left_knuckle.stl" />
+                    <mesh filename="package://robotiq_description/meshes/visual/left_knuckle.dae" />
+                </geometry>
+            </visual>
+            <collision>
+                <geometry>
+                    <mesh filename="package://robotiq_description/meshes/collision/left_knuckle.stl" />
                 </geometry>
             </collision>
@@ -61,10 +61,10 @@
             <visual>
                 <geometry>
-                    <mesh filename="file://$(find robotiq_description)/meshes/visual/right_knuckle.dae" />
-                </geometry>
-            </visual>
-            <collision>
-                <geometry>
-                    <mesh filename="file://$(find robotiq_description)/meshes/collision/right_knuckle.stl" />
+                    <mesh filename="package://robotiq_description/meshes/visual/right_knuckle.dae" />
+                </geometry>
+            </visual>
+            <collision>
+                <geometry>
+                    <mesh filename="package://robotiq_description/meshes/collision/right_knuckle.stl" />
                 </geometry>
             </collision>
@@ -78,10 +78,10 @@
             <visual>
                 <geometry>
-                    <mesh filename="file://$(find robotiq_description)/meshes/visual/left_finger.dae" />
-                </geometry>
-            </visual>
-            <collision>
-                <geometry>
-                    <mesh filename="file://$(find robotiq_description)/meshes/collision/left_finger.stl" />
+                    <mesh filename="package://robotiq_description/meshes/visual/left_finger.dae" />
+                </geometry>
+            </visual>
+            <collision>
+                <geometry>
+                    <mesh filename="package://robotiq_description/meshes/collision/left_finger.stl" />
                 </geometry>
             </collision>
@@ -95,10 +95,10 @@
             <visual>
                 <geometry>
-                    <mesh filename="file://$(find robotiq_description)/meshes/visual/right_finger.dae" />
-                </geometry>
-            </visual>
-            <collision>
-                <geometry>
-                    <mesh filename="file://$(find robotiq_description)/meshes/collision/right_finger.stl" />
+                    <mesh filename="package://robotiq_description/meshes/visual/right_finger.dae" />
+                </geometry>
+            </visual>
+            <collision>
+                <geometry>
+                    <mesh filename="package://robotiq_description/meshes/collision/right_finger.stl" />
                 </geometry>
             </collision>
@@ -112,10 +112,10 @@
             <visual>
                 <geometry>
-                    <mesh filename="file://$(find robotiq_description)/meshes/visual/left_inner_knuckle.dae" />
-                </geometry>
-            </visual>
-            <collision>
-                <geometry>
-                    <mesh filename="file://$(find robotiq_description)/meshes/collision/left_inner_knuckle.stl" />
+                    <mesh filename="package://robotiq_description/meshes/visual/left_inner_knuckle.dae" />
+                </geometry>
+            </visual>
+            <collision>
+                <geometry>
+                    <mesh filename="package://robotiq_description/meshes/collision/left_inner_knuckle.stl" />
                 </geometry>
             </collision>
@@ -129,10 +129,10 @@
             <visual>
                 <geometry>
-                    <mesh filename="file://$(find robotiq_description)/meshes/visual/right_inner_knuckle.dae" />
-                </geometry>
-            </visual>
-            <collision>
-                <geometry>
-                    <mesh filename="file://$(find robotiq_description)/meshes/collision/right_inner_knuckle.stl" />
+                    <mesh filename="package://robotiq_description/meshes/visual/right_inner_knuckle.dae" />
+                </geometry>
+            </visual>
+            <collision>
+                <geometry>
+                    <mesh filename="package://robotiq_description/meshes/collision/right_inner_knuckle.stl" />
                 </geometry>
             </collision>
@@ -146,10 +146,10 @@
             <visual>
                 <geometry>
-                    <mesh filename="file://$(find robotiq_description)/meshes/visual/left_finger_tip.dae" />
-                </geometry>
-            </visual>
-            <collision>
-                <geometry>
-                    <mesh filename="file://$(find robotiq_description)/meshes/collision/left_finger_tip.stl" />
+                    <mesh filename="package://robotiq_description/meshes/visual/left_finger_tip.dae" />
+                </geometry>
+            </visual>
+            <collision>
+                <geometry>
+                    <mesh filename="package://robotiq_description/meshes/collision/left_finger_tip.stl" />
                 </geometry>
                 <surface>
@@ -181,10 +181,10 @@
             <visual>
                 <geometry>
-                    <mesh filename="file://$(find robotiq_description)/meshes/visual/right_finger_tip.dae" />
-                </geometry>
-            </visual>
-            <collision>
-                <geometry>
-                    <mesh filename="file://$(find robotiq_description)/meshes/collision/right_finger_tip.stl" />
+                    <mesh filename="package://robotiq_description/meshes/visual/right_finger_tip.dae" />
+                </geometry>
+            </visual>
+            <collision>
+                <geometry>
+                    <mesh filename="package://robotiq_description/meshes/collision/right_finger_tip.stl" />
                 </geometry>
                 <surface>
