Commit message: update 140 to match 85 gripper (#1)

File: robotiq_description/urdf/robotiq_2f_140.xacro (robot description, xacro)
@@ -17,5 +17,5 @@
         <origin xyz="0 0 0" rpy="0 0 0" />
         <geometry>
-          <mesh filename="package://robotiq_description/meshes/visual/2f_140/robotiq_arg2f_${stroke}_outer_knuckle.stl" />
+          <mesh filename="file://$(find robotiq_description)/meshes/visual/2f_140/robotiq_2f_${stroke}_outer_knuckle.stl" />
         </geometry>
         <material name="">
@@ -26,5 +26,5 @@
         <origin xyz="0 0 0" rpy="0 0 0" />
         <geometry>
-          <mesh filename="package://robotiq_description/meshes/collision/2f_140/robotiq_arg2f_${stroke}_outer_knuckle.stl" />
+          <mesh filename="file://$(find robotiq_description)/meshes/collision/2f_140/robotiq_2f_${stroke}_outer_knuckle.stl" />
         </geometry>
       </collision>
@@ -47,5 +47,5 @@
         <origin xyz="0 0 0" rpy="0 0 0" />
         <geometry>
-          <mesh filename="package://robotiq_description/meshes/visual/2f_140/robotiq_arg2f_${stroke}_outer_finger.stl" />
+          <mesh filename="file://$(find robotiq_description)/meshes/visual/2f_140/robotiq_2f_${stroke}_outer_finger.stl" />
         </geometry>
         <material name="">
@@ -56,5 +56,5 @@
         <origin xyz="0 0 0" rpy="0 0 0" />
         <geometry>
-          <mesh filename="package://robotiq_description/meshes/collision/2f_140/robotiq_arg2f_${stroke}_outer_finger.stl" />
+          <mesh filename="file://$(find robotiq_description)/meshes/collision/2f_140/robotiq_2f_${stroke}_outer_finger.stl" />
         </geometry>
       </collision>
@@ -77,5 +77,5 @@
         <origin xyz="0 0 0" rpy="0 0 0" />
         <geometry>
-          <mesh filename="package://robotiq_description/meshes/visual/2f_140/robotiq_arg2f_${stroke}_inner_knuckle.stl" />
+          <mesh filename="file://$(find robotiq_description)/meshes/visual/2f_140/robotiq_2f_${stroke}_inner_knuckle.stl" />
         </geometry>
         <material name="">
@@ -86,5 +86,5 @@
         <origin xyz="0 0 0" rpy="0 0 0" />
         <geometry>
-          <mesh filename="package://robotiq_description/meshes/collision/2f_140/robotiq_arg2f_${stroke}_inner_knuckle.stl" />
+          <mesh filename="file://$(find robotiq_description)/meshes/collision/2f_140/robotiq_2f_${stroke}_inner_knuckle.stl" />
         </geometry>
       </collision>
@@ -107,5 +107,5 @@
         <origin xyz="0 0 0" rpy="0 0 0" />
         <geometry>
-          <mesh filename="package://robotiq_description/meshes/visual/2f_140/robotiq_arg2f_${stroke}_inner_finger.stl" />
+          <mesh filename="file://$(find robotiq_description)/meshes/visual/2f_140/robotiq_2f_${stroke}_inner_finger.stl" />
         </geometry>
         <material name="">
@@ -116,5 +116,5 @@
         <origin xyz="0 0 0" rpy="0 0 0" />
         <geometry>
-          <mesh filename="package://robotiq_description/meshes/collision/2f_140/robotiq_arg2f_${stroke}_inner_finger.stl" />
+          <mesh filename="file://$(find robotiq_description)/meshes/collision/2f_140/robotiq_2f_${stroke}_inner_finger.stl" />
         </geometry>
       </collision>
@@ -143,4 +143,25 @@
       </collision>
     </link>
+  </xacro:macro>
+  <xacro:macro name="finger_joint" params="prefix">
+    <joint name="${prefix}finger_joint" type="revolute">
+      <origin xyz="0 -0.030601 0.054905" rpy="${pi / 2 + .725} 0 0" />
+      <parent link="${prefix}robotiq_140_base_link" />
+      <child link="${prefix}left_outer_knuckle" />
+      <axis xyz="-1 0 0" />
+      <limit lower="0" upper="0.7" velocity="2.0" effort="1000" />
+    </joint>
+    <xacro:finger_joints prefix="${prefix}" fingerprefix="left" reflect="1.0"/>
+  </xacro:macro>
+  <xacro:macro name="right_outer_knuckle_joint" params="prefix">
+    <joint name="${prefix}right_outer_knuckle_joint" type="revolute">
+      <origin xyz="0 0.030601 0.054905" rpy="${pi / 2 + .725} 0 ${pi}" />
+      <parent link="${prefix}robotiq_140_base_link" />
+      <child link="${prefix}right_outer_knuckle" />
+      <axis xyz="1 0 0" />
+      <limit lower="-0.725" upper="0.725" velocity="2.0" effort="1000" />
+    <mimic joint="${prefix}finger_joint" multiplier="-1" offset="0" />
+    </joint>
+    <xacro:finger_joints prefix="${prefix}" fingerprefix="right" reflect="-1.0"/>
   </xacro:macro>
   <xacro:macro name="outer_finger_joint" params="prefix fingerprefix">
@@ -155,5 +176,5 @@
     <joint name="${prefix}${fingerprefix}_inner_knuckle_joint" type="revolute">
       <origin xyz="0 ${reflect * -0.0127} 0.06142" rpy="${pi / 2 + .725} 0 ${(reflect - 1) * pi / 2}" />
-      <parent link="${prefix}robotiq_arg2f_base_link" />
+      <parent link="${prefix}robotiq_140_base_link" />
       <child link="${prefix}${fingerprefix}_inner_knuckle" />
       <axis xyz="1 0 0" />
@@ -180,34 +201,16 @@
     </joint>
   </xacro:macro>
-  <xacro:include filename="$(find robotiq_description)/urdf/robotiq_arg2f_140.xacro" />
-  <xacro:macro name="finger_joint" params="prefix">
-    <joint name="${prefix}finger_joint" type="revolute">
-      <origin xyz="0 -0.030601 0.054905" rpy="${pi / 2 + .725} 0 0" />
-      <parent link="${prefix}robotiq_arg2f_base_link" />
-      <child link="${prefix}left_outer_knuckle" />
-      <axis xyz="-1 0 0" />
-      <limit lower="0" upper="0.7" velocity="2.0" effort="1000" />
-    </joint>
-    <xacro:finger_joints prefix="${prefix}" fingerprefix="left" reflect="1.0"/>
-  </xacro:macro>
-  <xacro:macro name="right_outer_knuckle_joint" params="prefix">
-    <joint name="${prefix}right_outer_knuckle_joint" type="revolute">
-      <origin xyz="0 0.030601 0.054905" rpy="${pi / 2 + .725} 0 ${pi}" />
-      <parent link="${prefix}robotiq_arg2f_base_link" />
-      <child link="${prefix}right_outer_knuckle" />
-      <axis xyz="1 0 0" />
-      <limit lower="-0.725" upper="0.725" velocity="2.0" effort="1000" />
-    <mimic joint="${prefix}finger_joint" multiplier="-1" offset="0" />
-    </joint>
-    <xacro:finger_joints prefix="${prefix}" fingerprefix="right" reflect="-1.0"/>
-  </xacro:macro>
-  <xacro:macro name="robotiq_2f_140" params="prefix parent *origin">
-    <xacro:robotiq_arg2f_base_link prefix="${prefix}" parent="${parent}">
-      <xacro:insert_block name="origin"/>
-    </xacro:robotiq_arg2f_base_link>
-    <xacro:finger_links prefix="${prefix}" fingerprefix="left" stroke="140"/>
-    <xacro:finger_links prefix="${prefix}" fingerprefix="right" stroke="140"/>
-    <xacro:finger_joint prefix="${prefix}"/>
-    <xacro:right_outer_knuckle_joint prefix="${prefix}"/>
+  <xacro:macro name="finger_joints" params="prefix fingerprefix reflect">
+    <xacro:outer_finger_joint prefix="${prefix}" fingerprefix="${fingerprefix}"/>
+    <xacro:inner_knuckle_joint prefix="${prefix}" fingerprefix="${fingerprefix}" reflect="${reflect}"/>
+    <xacro:inner_finger_joint prefix="${prefix}" fingerprefix="${fingerprefix}"/>
+    <xacro:inner_finger_pad_joint prefix="${prefix}" fingerprefix="${fingerprefix}"/>
+  </xacro:macro>
+  <xacro:macro name="finger_links" params="prefix fingerprefix stroke">
+    <xacro:outer_knuckle prefix="${prefix}" fingerprefix="${fingerprefix}" stroke="${stroke}"/>
+    <xacro:outer_finger prefix="${prefix}" fingerprefix="${fingerprefix}" stroke="${stroke}"/>
+    <xacro:inner_finger prefix="${prefix}" fingerprefix="${fingerprefix}" stroke="${stroke}"/>
+    <xacro:inner_finger_pad prefix="${prefix}" fingerprefix="${fingerprefix}"/>
+    <xacro:inner_knuckle prefix="${prefix}" fingerprefix="${fingerprefix}" stroke="${stroke}"/>
   </xacro:macro>
 </robot>
