Commit message: add dummy link to rotate 2f-140 to match 2f-85

File: robotiq_description/urdf/2f_140.ros2_control.xacro (robot description, xacro)
@@ -13,5 +13,5 @@
             <hardware>
                 <xacro:if value="${sim_isaac}">
-                    <plugin>isaac_ros2_control/IsaacSystem</plugin>
+                    <plugin>topic_based_ros2_control/TopicBasedSystem</plugin>
                     <param name="joint_commands_topic">/isaac_joint_commands</param>
                     <param name="joint_states_topic">/isaac_joint_states</param>

File: robotiq_description/urdf/robotiq_2f_140_macro.urdf.xacro (robot description, xacro)
@@ -24,4 +24,11 @@
                 com_port="${com_port}"/>
         </xacro:if>
+        <!-- this is a temporary link to rotate the 2f-140 gripper to match the 2f-85 -->
+        <link name="${prefix}robotiq_base_link"/>
+        <joint name="${prefix}robotiq_base_joint" type="fixed">
+          <parent link="${parent}" />
+          <child link="${prefix}robotiq_base_link" />
+          <origin xyz="0 0 0" rpy="0 0 ${pi/2}" />
+        </joint>
         <link name="${prefix}robotiq_140_base_link">
         <inertial>
@@ -47,5 +54,5 @@
       </link>
       <joint name="${prefix}robotiq_140_base_joint" type="fixed">
-          <parent link="${parent}" />
+          <parent link="${prefix}robotiq_base_link" />
           <child link="${prefix}robotiq_140_base_link" />
           <xacro:insert_block name="origin" />
