Commit message: add child parent as params
Signed-off-by: Paul Gesel <paulgesel@gmail.com>

File: robotiq_description/urdf/ur_to_robotiq_adapter.urdf.xacro (robot description, xacro)
@@ -1,8 +1,8 @@
 <?xml version="1.0" encoding="utf-8"?>
 <robot xmlns:xacro="http://ros.org/wiki/xacro">
-  <xacro:macro name="ur_to_robotiq" params="prefix connected_to rotation:=^|${0.0}">
+  <xacro:macro name="ur_to_robotiq" params="prefix parent child rotation:=^|${0.0}">
     <joint name="${prefix}ur_to_robotiq_joint" type="fixed">
       <!-- The parent link must be read from the robot model it is attached to. -->
-      <parent link="${connected_to}"/>
+      <parent link="${parent}"/>
       <child link="${prefix}ur_to_robotiq_link"/>
       <origin xyz="0 0 0" rpy="0 0 ${rotation}"/>
@@ -29,9 +29,9 @@
     <joint name="${prefix}gripper_side_joint" type="fixed">
       <parent link="${prefix}ur_to_robotiq_link"/>
-      <child link="${prefix}gripper_mount_link"/>
+      <child link="${child}"/>
       <!-- <origin xyz="0 0 0.011" rpy="0 ${-pi/2} ${pi/2}"/> -->
       <origin xyz="0 0 0.011" rpy="0 0 0"/>
     </joint>
-    <link name="${prefix}gripper_mount_link"/>
+    <link name="${child}"/>
   </xacro:macro>
 </robot>

Commit message: use find

File: robotiq_description/urdf/ur_to_robotiq_adapter.urdf.xacro (robot description, xacro)
@@ -12,5 +12,5 @@
           <origin xyz="0 0 0" rpy="0 0 0" />
           <geometry>
-            <mesh filename="package://robotiq_description/meshes/visual/2f_85/ur_to_robotiq_adapter.dae"/>
+            <mesh filename="file://$(find robotiq_description)/meshes/visual/2f_85/ur_to_robotiq_adapter.dae"/>
           </geometry>
         </visual>
@@ -18,5 +18,5 @@
           <origin xyz="0 0 0" rpy="0 0 0"/>
           <geometry>
-            <mesh filename="package://robotiq_description/meshes/collision/2f_85/ur_to_robotiq_adapter.stl"/>
+            <mesh filename="file://$(find robotiq_description)/meshes/collision/2f_85/ur_to_robotiq_adapter.stl"/>
           </geometry>
         </collision>
