Commit message: Unify 2F_85 and 2F_140 link names

File: robotiq_description/urdf/2f_85.ros2_control.xacro (robot description, xacro)
@@ -40,5 +40,5 @@
             <!-- Joint interfaces -->
             <!-- With Gazebo or Hardware, they handle mimic joints, so we only need this command interface activated -->
-            <joint name="${prefix}robotiq_85_left_knuckle_joint">
+            <joint name="${prefix}left_knuckle_joint">
                 <command_interface name="position" />
                 <state_interface name="position">
@@ -49,5 +49,5 @@
             <!-- When simulating we need to include the rest of the gripper joints -->
             <xacro:if value="${use_fake_hardware or sim_isaac or sim_gazebo}">
-                <joint name="${prefix}robotiq_85_right_knuckle_joint">
+                <joint name="${prefix}right_knuckle_joint">
                     <xacro:unless value="${sim_gazebo}">
                         <state_interface name="position"/>
@@ -55,5 +55,5 @@
                     </xacro:unless>
                 </joint>
-                <joint name="${prefix}robotiq_85_left_inner_knuckle_joint">
+                <joint name="${prefix}left_inner_knuckle_joint">
                     <xacro:unless value="${sim_gazebo}">
                         <state_interface name="position"/>
@@ -61,5 +61,5 @@
                     </xacro:unless>
                 </joint>
-                <joint name="${prefix}robotiq_85_right_inner_knuckle_joint">
+                <joint name="${prefix}right_inner_knuckle_joint">
                     <xacro:unless value="${sim_gazebo}">
                         <state_interface name="position"/>
@@ -67,5 +67,5 @@
                     </xacro:unless>
                 </joint>
-                <joint name="${prefix}robotiq_85_left_finger_tip_joint">
+                <joint name="${prefix}left_finger_tip_joint">
                     <xacro:unless value="${sim_gazebo}">
                         <state_interface name="position"/>
@@ -73,5 +73,5 @@
                     </xacro:unless>
                 </joint>
-                <joint name="${prefix}robotiq_85_right_finger_tip_joint">
+                <joint name="${prefix}right_finger_tip_joint">
                     <xacro:unless value="${sim_gazebo}">
                         <state_interface name="position"/>

File: robotiq_description/urdf/robotiq_2f_85_macro.urdf.xacro (robot description, xacro)
@@ -28,5 +28,5 @@
                 com_port="${com_port}"/>
         </xacro:if>
-        <link name="${prefix}robotiq_85_base_link">
+        <link name="${prefix}robotiq_base_link">
             <visual>
                 <geometry>
@@ -45,5 +45,5 @@
             </inertial>
         </link>
-        <link name="${prefix}robotiq_85_left_knuckle_link">
+        <link name="${prefix}left_knuckle_link">
             <visual>
                 <geometry>
@@ -62,5 +62,5 @@
             </inertial>
         </link>
-        <link name="${prefix}robotiq_85_right_knuckle_link">
+        <link name="${prefix}right_knuckle_link">
             <visual>
                 <geometry>
@@ -79,5 +79,5 @@
             </inertial>
         </link>
-        <link name="${prefix}robotiq_85_left_finger_link">
+        <link name="${prefix}left_finger_link">
             <visual>
                 <geometry>
@@ -96,5 +96,5 @@
             </inertial>
         </link>
-        <link name="${prefix}robotiq_85_right_finger_link">
+        <link name="${prefix}right_finger_link">
             <visual>
                 <geometry>
@@ -113,5 +113,5 @@
             </inertial>
         </link>
-        <link name="${prefix}robotiq_85_left_inner_knuckle_link">
+        <link name="${prefix}left_inner_knuckle_link">
             <visual>
                 <geometry>
@@ -130,5 +130,5 @@
             </inertial>
         </link>
-        <link name="${prefix}robotiq_85_right_inner_knuckle_link">
+        <link name="${prefix}right_inner_knuckle_link">
             <visual>
                 <geometry>
@@ -147,5 +147,5 @@
             </inertial>
         </link>
-        <link name="${prefix}robotiq_85_left_finger_tip_link">
+        <link name="${prefix}left_finger_tip_link">
             <visual>
                 <geometry>
@@ -182,5 +182,5 @@
             </inertial>
         </link>
-        <link name="${prefix}robotiq_85_right_finger_tip_link">
+        <link name="${prefix}right_finger_tip_link">
             <visual>
                 <geometry>
@@ -217,61 +217,61 @@
             </inertial>
         </link>
-        <joint name="${prefix}robotiq_85_base_joint" type="fixed">
+        <joint name="${prefix}base_joint" type="fixed">
             <parent link="${parent}" />
-            <child link="${prefix}robotiq_85_base_link" />
+            <child link="${prefix}robotiq_base_link" />
             <xacro:insert_block name="origin" />
         </joint>
-        <joint name="${prefix}robotiq_85_left_knuckle_joint" type="revolute">
-            <parent link="${prefix}robotiq_85_base_link" />
-            <child link="${prefix}robotiq_85_left_knuckle_link" />
+        <joint name="${prefix}left_knuckle_joint" type="revolute">
+            <parent link="${prefix}robotiq_base_link" />
+            <child link="${prefix}left_knuckle_link" />
             <axis xyz="0 -1 0" />
             <origin xyz="0.03060114 0.0 0.05490452" rpy="0 0 0" />
             <limit lower="0.0" upper="0.8" velocity="0.5" effort="50" />
         </joint>
-        <joint name="${prefix}robotiq_85_right_knuckle_joint" type="revolute">
-            <parent link="${prefix}robotiq_85_base_link" />
-            <child link="${prefix}robotiq_85_right_knuckle_link" />
+        <joint name="${prefix}right_knuckle_joint" type="revolute">
+            <parent link="${prefix}robotiq_base_link" />
+            <child link="${prefix}right_knuckle_link" />
             <axis xyz="0 -1 0" />
             <origin xyz="-0.03060114 0.0 0.05490452" rpy="0 0 0" />
             <limit lower="-0.8" upper="0.0" velocity="0.5" effort="50" />
-            <mimic joint="${prefix}robotiq_85_left_knuckle_joint" multiplier="-1" />
-        </joint>
-        <joint name="${prefix}robotiq_85_left_finger_joint" type="fixed">
-            <parent link="${prefix}robotiq_85_left_knuckle_link" />
-            <child link="${prefix}robotiq_85_left_finger_link" />
+            <mimic joint="${prefix}left_knuckle_joint" multiplier="-1" />
+        </joint>
+        <joint name="${prefix}left_finger_joint" type="fixed">
+            <parent link="${prefix}left_knuckle_link" />
+            <child link="${prefix}left_finger_link" />
             <origin xyz="0.03152616 0.0 -0.00376347" rpy="0 0 0" />
         </joint>
-        <joint name="${prefix}robotiq_85_right_finger_joint" type="fixed">
-            <parent link="${prefix}robotiq_85_right_knuckle_link" />
-            <child link="${prefix}robotiq_85_right_finger_link" />
+        <joint name="${prefix}right_finger_joint" type="fixed">
+            <parent link="${prefix}right_knuckle_link" />
+            <child link="${prefix}right_finger_link" />
             <origin xyz="-0.03152616 0.0 -0.00376347" rpy="0 0 0" />
         </joint>
-        <joint name="${prefix}robotiq_85_left_inner_knuckle_joint" type="continuous">
-            <parent link="${prefix}robotiq_85_base_link" />
-            <child link="${prefix}robotiq_85_left_inner_knuckle_link" />
+        <joint name="${prefix}left_inner_knuckle_joint" type="continuous">
+            <parent link="${prefix}robotiq_base_link" />
+            <child link="${prefix}left_inner_knuckle_link" />
             <axis xyz="0 -1 0" />
             <origin xyz="0.0127 0.0 0.06142" rpy="0 0 0" />
-            <mimic joint="${prefix}robotiq_85_left_knuckle_joint" />
-        </joint>
-        <joint name="${prefix}robotiq_85_right_inner_knuckle_joint" type="continuous">
-            <parent link="${prefix}robotiq_85_base_link" />
-            <child link="${prefix}robotiq_85_right_inner_knuckle_link" />
+            <mimic joint="${prefix}left_knuckle_joint" />
+        </joint>
+        <joint name="${prefix}right_inner_knuckle_joint" type="continuous">
+            <parent link="${prefix}robotiq_base_link" />
+            <child link="${prefix}right_inner_knuckle_link" />
             <axis xyz="0 -1 0" />
             <origin xyz="-0.0127 0.0 0.06142" rpy="0 0 0" />
-            <mimic joint="${prefix}robotiq_85_left_knuckle_joint" multiplier="-1" />
-        </joint>
-        <joint name="${prefix}robotiq_85_left_finger_tip_joint" type="continuous">
-            <parent link="${prefix}robotiq_85_left_finger_link" />
-            <child link="${prefix}robotiq_85_left_finger_tip_link" />
+            <mimic joint="${prefix}left_knuckle_joint" multiplier="-1" />
+        </joint>
+        <joint name="${prefix}left_finger_tip_joint" type="continuous">
+            <parent link="${prefix}left_finger_link" />
+            <child link="${prefix}left_finger_tip_link" />
             <axis xyz="0 -1 0" />
             <origin xyz="0.00563134 0.0 0.04718515" rpy="0 0 0" />
-            <mimic joint="${prefix}robotiq_85_left_knuckle_joint" multiplier="-1" />
-        </joint>
-        <joint name="${prefix}robotiq_85_right_finger_tip_joint" type="continuous">
-            <parent link="${prefix}robotiq_85_right_finger_link" />
-            <child link="${prefix}robotiq_85_right_finger_tip_link" />
+            <mimic joint="${prefix}left_knuckle_joint" multiplier="-1" />
+        </joint>
+        <joint name="${prefix}right_finger_tip_joint" type="continuous">
+            <parent link="${prefix}right_finger_link" />
+            <child link="${prefix}right_finger_tip_link" />
             <axis xyz="0 -1 0" />
             <origin xyz="-0.00563134 0.0 0.04718515" rpy="0 0 0" />
-            <mimic joint="${prefix}robotiq_85_left_knuckle_joint" />
+            <mimic joint="${prefix}left_knuckle_joint" />
         </joint>
     </xacro:macro>
