Commit message: Adjust frames position and origins

File: robotiq_description/urdf/robotiq_hande_macro.urdf.xacro (robot description, xacro)
@@ -88,5 +88,5 @@
           <link name="$(arg prefix)tcp_link"/>
           <joint name="$(arg prefix)tcp_link_joint" type="fixed">
-            <origin xyz="0 0 0.125" rpy="0 0 0"/>
+            <origin xyz="0 0 0.125" rpy="0 0 -1.571"/>
             <parent link="$(arg prefix)hand_e_base_link"/>
             <child link="$(arg prefix)tcp_link"/>
@@ -95,5 +95,5 @@
           <link name="$(arg prefix)tcp_link_tube"/>
           <joint name="$(arg prefix)tcp_joint_tube" type="fixed">
-            <origin xyz="0 0 0" rpy="0 0 0"/>
+            <origin xyz="0 0 0" rpy="3.1416 0 -1.571"/>
             <parent link="$(arg prefix)tcp_link"/>
             <child link="$(arg prefix)tcp_link_tube"/>
@@ -102,5 +102,5 @@
           <link name="$(arg prefix)tcp_link_rack"/>
           <joint name="$(arg prefix)tcp_joint_rack" type="fixed">
-            <origin xyz="0 -0.0 0" rpy="0 0 0"/>
+            <origin xyz="0.035 0 0" rpy="3.1416 0 -1.571"/>
             <parent link="$(arg prefix)tcp_link"/>
             <child link="$(arg prefix)tcp_link_rack"/>
