Commit message: remove custom tcp links

File: robotiq_description/urdf/robotiq_hand_e_macro.urdf.xacro (robot description, xacro)
@@ -98,5 +98,4 @@
         <mimic joint="${prefix}hande_finger_distance" multiplier="-0.5" offset="${gripper_maximal_stroke/2}"/>
       </joint>
-      <!-- TODO (Manuel) Remove this tmp tcp_link -->
       <link name="$(arg prefix)tcp_link"/>
       <joint name="$(arg prefix)tcp_link_joint" type="fixed">
@@ -105,18 +104,4 @@
         <child link="$(arg prefix)tcp_link"/>
       </joint>
-      <!-- TCP Link Tube -->
-      <link name="$(arg prefix)tcp_link_tube"/>
-      <joint name="$(arg prefix)tcp_joint_tube" type="fixed">
-        <origin xyz="0 0 0" rpy="${pi} 0 ${-pi/2}"/>
-        <parent link="$(arg prefix)tcp_link"/>
-        <child link="$(arg prefix)tcp_link_tube"/>
-      </joint>
-      <!-- TCP Link Rack -->
-      <link name="$(arg prefix)tcp_link_rack"/>
-      <joint name="$(arg prefix)tcp_joint_rack" type="fixed">
-        <origin xyz="0.035 0 0" rpy="${pi} 0 ${-pi/2}"/>
-        <parent link="$(arg prefix)tcp_link"/>
-        <child link="$(arg prefix)tcp_link_rack"/>
-      </joint>
     </xacro:macro>
 </robot>

Commit message: quick and dirty adaption to new gripper size

File: robotiq_description/urdf/robotiq_hand_e_macro.urdf.xacro (robot description, xacro)
@@ -11,4 +11,8 @@
     <xacro:macro name="robotiq_hande" params="prefix parent *origin">
       <xacro:property name="gripper_maximal_stroke" value="0.050" />
+      <!-- TODO adapt mesh and collision of gripper and remove scaling -->
+      <xacro:property name="gripper_scale_x" value="1.0" />
+      <xacro:property name="gripper_scale_y" value="${8.5/6.2}" />
+      <xacro:property name="gripper_scale_z" value="${2.5/4.0}" />
       <link name="${prefix}hand_e_base_link">
           <inertial>
@@ -41,5 +45,5 @@
             <origin rpy="0 0 0" xyz="0 0 0"/>
             <geometry>
-              <mesh filename="package://robotiq_description/meshes/visual/hande/left_finger.dae" />
+              <mesh filename="package://robotiq_description/meshes/visual/hande/left_finger.dae" scale="${gripper_scale_x} ${gripper_scale_y} ${gripper_scale_z}"/>
             </geometry>
             <material name="gray">
@@ -50,5 +54,5 @@
             <origin rpy="0 0 0" xyz="0 0 0"/>
             <geometry>
-              <mesh filename="package://robotiq_description/meshes/collision/hande/left_finger.stl" />
+              <mesh filename="package://robotiq_description/meshes/collision/hande/left_finger.stl" scale="${gripper_scale_x} ${gripper_scale_y} ${gripper_scale_z}"/>
             </geometry>
           </collision>
@@ -58,5 +62,5 @@
             <origin rpy="0 0 0" xyz="0 0 0"/>
             <geometry>
-              <mesh filename="package://robotiq_description/meshes/visual/hande/right_finger.dae" />
+              <mesh filename="package://robotiq_description/meshes/visual/hande/right_finger.dae" scale="${gripper_scale_x} ${gripper_scale_y} ${gripper_scale_z}"/>
             </geometry>
             <material name="gray">
@@ -67,5 +71,5 @@
             <origin rpy="0 0 0" xyz="0 0 0"/>
             <geometry>
-              <mesh filename="package://robotiq_description/meshes/collision/hande/right_finger.stl" />
+              <mesh filename="package://robotiq_description/meshes/collision/hande/right_finger.stl" scale="${gripper_scale_x} ${gripper_scale_y} ${gripper_scale_z}"/>
             </geometry>
           </collision>
@@ -100,5 +104,5 @@
       <link name="$(arg prefix)tcp_link"/>
       <joint name="$(arg prefix)tcp_link_joint" type="fixed">
-        <origin xyz="0 0 0.125" rpy="0 0 ${-pi/2}"/>
+        <origin xyz="0 0 0.1125" rpy="0 0 ${-pi/2}"/>
         <parent link="$(arg prefix)hand_e_base_link"/>
         <child link="$(arg prefix)tcp_link"/>

Commit message: use visual for collision

File: robotiq_description/urdf/robotiq_hand_e_macro.urdf.xacro (robot description, xacro)
@@ -54,5 +54,5 @@
             <origin rpy="0 0 0" xyz="0 0 0"/>
             <geometry>
-              <mesh filename="package://robotiq_description/meshes/collision/hande/left_finger.stl" scale="${gripper_scale_x} ${gripper_scale_y} ${gripper_scale_z}"/>
+              <mesh filename="package://robotiq_description/meshes/visual/hande/left_finger.dae" scale="${gripper_scale_x} ${gripper_scale_y} ${gripper_scale_z}"/>
             </geometry>
           </collision>
@@ -71,5 +71,5 @@
             <origin rpy="0 0 0" xyz="0 0 0"/>
             <geometry>
-              <mesh filename="package://robotiq_description/meshes/collision/hande/right_finger.stl" scale="${gripper_scale_x} ${gripper_scale_y} ${gripper_scale_z}"/>
+              <mesh filename="package://robotiq_description/meshes/visual/hande/right_finger.dae" scale="${gripper_scale_x} ${gripper_scale_y} ${gripper_scale_z}"/>
             </geometry>
           </collision>

Commit message: Added default finger meshes and created parameters for the macro of the gripper

File: robotiq_description/urdf/robotiq_hand_e_macro.urdf.xacro (robot description, xacro)
@@ -9,5 +9,8 @@
     </material>
     <!-- Gripper macro hand-e -->
-    <xacro:macro name="robotiq_hande" params="prefix parent *origin">
+    <xacro:macro name="robotiq_hande" params="prefix parent
+    right_finger:=default_right right_finger_coll:=default_right_coll left_finger:=default_left  left_finger_coll:=default_left_coll
+    *origin">
+      <xacro:property name="file_path" value="file://$(find robotiq_description)" />
       <xacro:property name="gripper_maximal_stroke" value="0.050" />
       <!-- TODO adapt mesh and collision of gripper and remove scaling -->
@@ -24,5 +27,5 @@
               <origin rpy="0 0 0" xyz="0 0 0"/>
               <geometry>
-                  <mesh filename="package://robotiq_description/meshes/visual/hande/hand-e.dae" scale="1.0 1.0 1.0"/>
+                  <mesh filename="${file_path}/meshes/visual/hande/hand-e.dae" scale="1.0 1.0 1.0"/>
               </geometry>
               <material name="dark" />
@@ -31,5 +34,5 @@
               <origin rpy="0 0 0" xyz="0 0 0"/>
               <geometry>
-                  <mesh filename="package://robotiq_description/meshes/collision/hande/hand-e.stl" scale="1.0 1.0 1.0"/>
+                  <mesh filename="${file_path}/meshes/collision/hande/hand-e.stl" scale="1.0 1.0 1.0"/>
               </geometry>
           </collision>
@@ -45,5 +48,10 @@
             <origin rpy="0 0 0" xyz="0 0 0"/>
             <geometry>
-              <mesh filename="package://robotiq_description/meshes/visual/hande/left_finger.dae" scale="${gripper_scale_x} ${gripper_scale_y} ${gripper_scale_z}"/>
+              <xacro:if value="${left_finger == 'default_left'}">
+                  <mesh filename="${file_path}/meshes/visual/hande/left_finger.dae" />
+              </xacro:if>
+              <xacro:if value="${left_finger != 'default_left'}">
+                  <mesh filename="${left_finger}" />
+              </xacro:if>
             </geometry>
             <material name="gray">
@@ -54,5 +62,10 @@
             <origin rpy="0 0 0" xyz="0 0 0"/>
             <geometry>
-              <mesh filename="package://robotiq_description/meshes/visual/hande/left_finger.dae" scale="${gripper_scale_x} ${gripper_scale_y} ${gripper_scale_z}"/>
+              <xacro:if value="${left_finger_coll == 'default_left_coll'}">
+                  <mesh filename="${file_path}/meshes/collision/hande/left_finger.stl" />
+              </xacro:if>
+              <xacro:if value="${left_finger_coll != 'default_left_coll'}">
+                  <mesh filename="${left_finger_coll}" />
+              </xacro:if>
             </geometry>
           </collision>
@@ -62,5 +75,10 @@
             <origin rpy="0 0 0" xyz="0 0 0"/>
             <geometry>
-              <mesh filename="package://robotiq_description/meshes/visual/hande/right_finger.dae" scale="${gripper_scale_x} ${gripper_scale_y} ${gripper_scale_z}"/>
+              <xacro:if value="${right_finger == 'default_right'}">
+                  <mesh filename="${file_path}/meshes/visual/hande/right_finger.dae" />
+              </xacro:if>
+              <xacro:if value="${right_finger != 'default_right'}">
+                  <mesh filename="${right_finger}" />
+              </xacro:if>
             </geometry>
             <material name="gray">
@@ -71,5 +89,10 @@
             <origin rpy="0 0 0" xyz="0 0 0"/>
             <geometry>
-              <mesh filename="package://robotiq_description/meshes/visual/hande/right_finger.dae" scale="${gripper_scale_x} ${gripper_scale_y} ${gripper_scale_z}"/>
+              <xacro:if value="${right_finger_coll == 'default_right_coll'}">
+                  <mesh filename="${file_path}/meshes/collision/hande/right_finger.stl" />
+              </xacro:if>
+              <xacro:if value="${right_finger_coll != 'default_right_coll'}">
+                  <mesh filename="${right_finger_coll}" />
+              </xacro:if>
             </geometry>
           </collision>

Commit message: Adjusted macro to support the scaling of meshes and shifting of grippers tcp in z direction.

File: robotiq_description/urdf/robotiq_hand_e_macro.urdf.xacro (robot description, xacro)
@@ -9,13 +9,31 @@
     </material>
     <!-- Gripper macro hand-e -->
-    <xacro:macro name="robotiq_hande" params="prefix parent
-    right_finger:=default_right right_finger_coll:=default_right_coll left_finger:=default_left  left_finger_coll:=default_left_coll
-    *origin">
+    <xacro:macro name="robotiq_hande" params="
+                 prefix parent *origin
+                 left_finger_visual:=default left_finger_collision:=default left_finger_scale:=default
+                 right_finger_visual:=default right_finger_collision:=default right_finger_scale:=default
+                 tcp_z_offset:=0.1325
+                 ">
       <xacro:property name="file_path" value="file://$(find robotiq_description)" />
       <xacro:property name="gripper_maximal_stroke" value="0.050" />
-      <!-- TODO adapt mesh and collision of gripper and remove scaling -->
-      <xacro:property name="gripper_scale_x" value="1.0" />
-      <xacro:property name="gripper_scale_y" value="${8.5/6.2}" />
-      <xacro:property name="gripper_scale_z" value="${2.5/4.0}" />
+      <!-- resolve complex default values -->
+      <xacro:if value="${left_finger_visual == 'default'}">
+        <xacro:property name="left_finger_visual" value="${file_path}/meshes/visual/hande/left_finger.dae" />
+      </xacro:if>
+      <xacro:if value="${left_finger_collision == 'default'}">
+        <xacro:property name="left_finger_collision" value="${file_path}/meshes/collision/hande/left_finger.stl" />
+      </xacro:if>
+      <xacro:if value="${left_finger_scale == 'default'}">
+        <xacro:property name="left_finger_scale" value="1.0 1.0 1.0" />
+      </xacro:if>
+      <xacro:if value="${right_finger_visual == 'default'}">
+        <xacro:property name="right_finger_visual" value="${file_path}/meshes/visual/hande/right_finger.dae" />
+      </xacro:if>
+      <xacro:if value="${right_finger_collision == 'default'}">
+        <xacro:property name="right_finger_collision" value="${file_path}/meshes/collision/hande/right_finger.stl" />
+      </xacro:if>
+      <xacro:if value="${right_finger_scale == 'default'}">
+        <xacro:property name="right_finger_scale" value="1.0 1.0 1.0" />
+      </xacro:if>
       <link name="${prefix}hand_e_base_link">
           <inertial>
@@ -48,10 +66,5 @@
             <origin rpy="0 0 0" xyz="0 0 0"/>
             <geometry>
-              <xacro:if value="${left_finger == 'default_left'}">
-                  <mesh filename="${file_path}/meshes/visual/hande/left_finger.dae" />
-              </xacro:if>
-              <xacro:if value="${left_finger != 'default_left'}">
-                  <mesh filename="${left_finger}" />
-              </xacro:if>
+              <mesh filename="${left_finger_visual}" scale="${left_finger_scale}" />
             </geometry>
             <material name="gray">
@@ -62,10 +75,5 @@
             <origin rpy="0 0 0" xyz="0 0 0"/>
             <geometry>
-              <xacro:if value="${left_finger_coll == 'default_left_coll'}">
-                  <mesh filename="${file_path}/meshes/collision/hande/left_finger.stl" />
-              </xacro:if>
-              <xacro:if value="${left_finger_coll != 'default_left_coll'}">
-                  <mesh filename="${left_finger_coll}" />
-              </xacro:if>
+              <mesh filename="${left_finger_collision}" scale="${left_finger_scale}" />
             </geometry>
           </collision>
@@ -75,10 +83,5 @@
             <origin rpy="0 0 0" xyz="0 0 0"/>
             <geometry>
-              <xacro:if value="${right_finger == 'default_right'}">
-                  <mesh filename="${file_path}/meshes/visual/hande/right_finger.dae" />
-              </xacro:if>
-              <xacro:if value="${right_finger != 'default_right'}">
-                  <mesh filename="${right_finger}" />
-              </xacro:if>
+              <mesh filename="${right_finger_visual}" scale="${right_finger_scale}" />
             </geometry>
             <material name="gray">
@@ -89,10 +92,5 @@
             <origin rpy="0 0 0" xyz="0 0 0"/>
             <geometry>
-              <xacro:if value="${right_finger_coll == 'default_right_coll'}">
-                  <mesh filename="${file_path}/meshes/collision/hande/right_finger.stl" />
-              </xacro:if>
-              <xacro:if value="${right_finger_coll != 'default_right_coll'}">
-                  <mesh filename="${right_finger_coll}" />
-              </xacro:if>
+              <mesh filename="${right_finger_collision}" scale="${right_finger_scale}" />
             </geometry>
           </collision>
@@ -127,5 +125,5 @@
       <link name="$(arg prefix)tcp_link"/>
       <joint name="$(arg prefix)tcp_link_joint" type="fixed">
-        <origin xyz="0 0 0.1125" rpy="0 0 ${-pi/2}"/>
+        <origin xyz="0 0 ${tcp_z_offset}" rpy="0 0 ${-pi/2}"/>
         <parent link="$(arg prefix)hand_e_base_link"/>
         <child link="$(arg prefix)tcp_link"/>

Commit message: Add primitive fingers for collision on the Robotiq Hand.

File: robotiq_description/urdf/robotiq_hand_e_macro.urdf.xacro (robot description, xacro)
@@ -11,6 +11,8 @@
     <xacro:macro name="robotiq_hande" params="
                  prefix parent *origin
-                 left_finger_visual:=default left_finger_collision:=default left_finger_scale:=default
-                 right_finger_visual:=default right_finger_collision:=default right_finger_scale:=default
+                 left_finger_visual:=default left_finger_collision:=default
+                 left_finger_scale:=default left_finger_collision_scale:=default
+                 right_finger_visual:=default right_finger_collision:=default
+                 right_finger_scale:=default right_finger_collision_scale:=default
                  tcp_z_offset:=0.1325
                  ">
@@ -27,4 +29,7 @@
         <xacro:property name="left_finger_scale" value="1.0 1.0 1.0" />
       </xacro:if>
+      <xacro:if value="${left_finger_collision_scale == 'default'}">
+        <xacro:property name="left_finger_collision_scale" value="1.0 1.0 1.0" />
+      </xacro:if>
       <xacro:if value="${right_finger_visual == 'default'}">
         <xacro:property name="right_finger_visual" value="${file_path}/meshes/visual/hande/right_finger.dae" />
@@ -33,6 +38,9 @@
         <xacro:property name="right_finger_collision" value="${file_path}/meshes/collision/hande/right_finger.stl" />
       </xacro:if>
-      <xacro:if value="${right_finger_scale == 'default'}">
+      <xacro:if value="${right_finger_collision_scale == 'default'}">
         <xacro:property name="right_finger_scale" value="1.0 1.0 1.0" />
+      </xacro:if>
+      <xacro:if value="${right_finger_collision_scale == 'default'}">
+        <xacro:property name="right_finger_collision_scale" value="1.0 1.0 1.0" />
       </xacro:if>
       <link name="${prefix}hand_e_base_link">
@@ -73,7 +81,8 @@
           </visual>
           <collision>
-            <origin rpy="0 0 0" xyz="0 0 0"/>
+            <origin rpy="0 0 0" xyz="${-0.010} ${-0.075/2} ${0.028/2}"/>
             <geometry>
-              <mesh filename="${left_finger_collision}" scale="${left_finger_scale}" />
+<!--               <mesh filename="${left_finger_collision}" scale="1.0 1.0 1.0" /> -->
+              <box size="${left_finger_collision_scale}" />
             </geometry>
           </collision>
@@ -90,7 +99,8 @@
           </visual>
           <collision>
-            <origin rpy="0 0 0" xyz="0 0 0"/>
+            <origin rpy="0 0 0" xyz="${0.010} ${-0.075/2} ${0.028/2}"/>
             <geometry>
-              <mesh filename="${right_finger_collision}" scale="${right_finger_scale}" />
+              <box size="${right_finger_collision_scale}" />
+<!--               <mesh filename="${right_finger_collision}" scale="1.0 1.0 1.0" /> -->
             </geometry>
           </collision>

Commit message: Use more exact collision mesh.

File: robotiq_description/urdf/robotiq_hand_e_macro.urdf.xacro (robot description, xacro)
@@ -61,4 +61,5 @@
               <geometry>
                   <mesh filename="${file_path}/meshes/collision/hande/hand-e.stl" scale="1.0 1.0 1.0"/>
+                  <!--<mesh filename="${file_path}/meshes/collision/hande/hand-e_convex_hull.stl" scale="1.0 1.0 1.0"/>-->
               </geometry>
           </collision>
