Commit message: Update meshes's file paths

File: robotiq_description/urdf/robotiq_2f_85_macro.urdf.xacro (robot description, xacro)
@@ -32,5 +32,5 @@
             <collision>
                 <geometry>
-                    <mesh filename="file://$(find robotiq_description)/meshes/collision/robotiq_base.stl" />
+                    <mesh filename="file://$(find robotiq_description)/meshes/collision/f2_85/robotiq_base.stl" />
                 </geometry>
             </collision>
@@ -49,5 +49,5 @@
             <collision>
                 <geometry>
-                    <mesh filename="file://$(find robotiq_description)/meshes/collision/left_knuckle.stl" />
+                    <mesh filename="file://$(find robotiq_description)/meshes/collision/f2_85/left_knuckle.stl" />
                 </geometry>
             </collision>
@@ -66,5 +66,5 @@
             <collision>
                 <geometry>
-                    <mesh filename="file://$(find robotiq_description)/meshes/collision/right_knuckle.stl" />
+                    <mesh filename="file://$(find robotiq_description)/meshes/collision/f2_85/right_knuckle.stl" />
                 </geometry>
             </collision>
@@ -83,5 +83,5 @@
             <collision>
                 <geometry>
-                    <mesh filename="file://$(find robotiq_description)/meshes/collision/left_finger.stl" />
+                    <mesh filename="file://$(find robotiq_description)/meshes/collision/f2_85/left_finger.stl" />
                 </geometry>
             </collision>
@@ -100,5 +100,5 @@
             <collision>
                 <geometry>
-                    <mesh filename="file://$(find robotiq_description)/meshes/collision/right_finger.stl" />
+                    <mesh filename="file://$(find robotiq_description)/meshes/collision/f2_85/right_finger.stl" />
                 </geometry>
             </collision>
@@ -117,5 +117,5 @@
             <collision>
                 <geometry>
-                    <mesh filename="file://$(find robotiq_description)/meshes/collision/left_inner_knuckle.stl" />
+                    <mesh filename="file://$(find robotiq_description)/meshes/collision/f2_85/left_inner_knuckle.stl" />
                 </geometry>
             </collision>
@@ -134,5 +134,5 @@
             <collision>
                 <geometry>
-                    <mesh filename="file://$(find robotiq_description)/meshes/collision/right_inner_knuckle.stl" />
+                    <mesh filename="file://$(find robotiq_description)/meshes/collision/f2_85/right_inner_knuckle.stl" />
                 </geometry>
             </collision>
@@ -151,5 +151,5 @@
             <collision>
                 <geometry>
-                    <mesh filename="file://$(find robotiq_description)/meshes/collision/left_finger_tip.stl" />
+                    <mesh filename="file://$(find robotiq_description)/meshes/collision/f2_85/left_finger_tip.stl" />
                 </geometry>
                 <surface>
@@ -186,5 +186,5 @@
             <collision>
                 <geometry>
-                    <mesh filename="file://$(find robotiq_description)/meshes/collision/right_finger_tip.stl" />
+                    <mesh filename="file://$(find robotiq_description)/meshes/collision/f2_85/right_finger_tip.stl" />
                 </geometry>
                 <surface>

File: robotiq_description/urdf/ur_to_robotiq_adapter.urdf.xacro (robot description, xacro)
@@ -18,5 +18,5 @@
           <origin xyz="0 0 0" rpy="0 0 0"/>
           <geometry>
-            <mesh filename="package://robotiq_description/meshes/collision/ur_to_robotiq_adapter.stl"/>
+            <mesh filename="package://robotiq_description/meshes/collision/f2_85/ur_to_robotiq_adapter.stl"/>
           </geometry>
         </collision>

Commit message: Fix typo f2 -> 2f

File: robotiq_description/urdf/robotiq_2f_85_macro.urdf.xacro (robot description, xacro)
@@ -13,5 +13,5 @@
         com_port:=/dev/ttyUSB0">
         <!-- ros2 control include -->
-        <xacro:include filename="$(find robotiq_description)/urdf/f2_85.ros2_control.xacro" />
+        <xacro:include filename="$(find robotiq_description)/urdf/2f_85.ros2_control.xacro" />
         <!-- if we are simulating or directly communicating with the gripper we need a ros2 control instance -->
         <xacro:if value="${include_ros2_control}">
@@ -32,5 +32,5 @@
             <collision>
                 <geometry>
-                    <mesh filename="file://$(find robotiq_description)/meshes/collision/f2_85/robotiq_base.stl" />
+                    <mesh filename="file://$(find robotiq_description)/meshes/collision/2f_85/robotiq_base.stl" />
                 </geometry>
             </collision>
@@ -49,5 +49,5 @@
             <collision>
                 <geometry>
-                    <mesh filename="file://$(find robotiq_description)/meshes/collision/f2_85/left_knuckle.stl" />
+                    <mesh filename="file://$(find robotiq_description)/meshes/collision/2f_85/left_knuckle.stl" />
                 </geometry>
             </collision>
@@ -66,5 +66,5 @@
             <collision>
                 <geometry>
-                    <mesh filename="file://$(find robotiq_description)/meshes/collision/f2_85/right_knuckle.stl" />
+                    <mesh filename="file://$(find robotiq_description)/meshes/collision/2f_85/right_knuckle.stl" />
                 </geometry>
             </collision>
@@ -83,5 +83,5 @@
             <collision>
                 <geometry>
-                    <mesh filename="file://$(find robotiq_description)/meshes/collision/f2_85/left_finger.stl" />
+                    <mesh filename="file://$(find robotiq_description)/meshes/collision/2f_85/left_finger.stl" />
                 </geometry>
             </collision>
@@ -100,5 +100,5 @@
             <collision>
                 <geometry>
-                    <mesh filename="file://$(find robotiq_description)/meshes/collision/f2_85/right_finger.stl" />
+                    <mesh filename="file://$(find robotiq_description)/meshes/collision/2f_85/right_finger.stl" />
                 </geometry>
             </collision>
@@ -117,5 +117,5 @@
             <collision>
                 <geometry>
-                    <mesh filename="file://$(find robotiq_description)/meshes/collision/f2_85/left_inner_knuckle.stl" />
+                    <mesh filename="file://$(find robotiq_description)/meshes/collision/2f_85/left_inner_knuckle.stl" />
                 </geometry>
             </collision>
@@ -134,5 +134,5 @@
             <collision>
                 <geometry>
-                    <mesh filename="file://$(find robotiq_description)/meshes/collision/f2_85/right_inner_knuckle.stl" />
+                    <mesh filename="file://$(find robotiq_description)/meshes/collision/2f_85/right_inner_knuckle.stl" />
                 </geometry>
             </collision>
@@ -151,5 +151,5 @@
             <collision>
                 <geometry>
-                    <mesh filename="file://$(find robotiq_description)/meshes/collision/f2_85/left_finger_tip.stl" />
+                    <mesh filename="file://$(find robotiq_description)/meshes/collision/2f_85/left_finger_tip.stl" />
                 </geometry>
                 <surface>
@@ -186,5 +186,5 @@
             <collision>
                 <geometry>
-                    <mesh filename="file://$(find robotiq_description)/meshes/collision/f2_85/right_finger_tip.stl" />
+                    <mesh filename="file://$(find robotiq_description)/meshes/collision/2f_85/right_finger_tip.stl" />
                 </geometry>
                 <surface>

File: robotiq_description/urdf/robotiq_arg2f_140.xacro (robot description, xacro)
@@ -11,5 +11,5 @@
         <origin xyz="0 0 0" rpy="0 0 0" />
         <geometry>
-          <mesh filename="package://robotiq_description/meshes/visual/f2_140/robotiq_arg2f_base_link.stl" />
+          <mesh filename="package://robotiq_description/meshes/visual/2f_140/robotiq_arg2f_base_link.stl" />
         </geometry>
         <material name="">
@@ -20,5 +20,5 @@
         <origin xyz="0 0 0" rpy="0 0 0" />
         <geometry>
-          <mesh filename="package://robotiq_description/meshes/collision/f2_140/robotiq_arg2f_base_link.stl" />
+          <mesh filename="package://robotiq_description/meshes/collision/2f_140/robotiq_arg2f_base_link.stl" />
         </geometry>
       </collision>

File: robotiq_description/urdf/robotiq_arg2f_140_model_macro.xacro (robot description, xacro)
@@ -17,5 +17,5 @@
         <origin xyz="0 0 0" rpy="0 0 0" />
         <geometry>
-          <mesh filename="package://robotiq_description/meshes/visual/f2_140/robotiq_arg2f_${stroke}_outer_knuckle.stl" />
+          <mesh filename="package://robotiq_description/meshes/visual/2f_140/robotiq_arg2f_${stroke}_outer_knuckle.stl" />
         </geometry>
         <material name="">
@@ -26,5 +26,5 @@
         <origin xyz="0 0 0" rpy="0 0 0" />
         <geometry>
-          <mesh filename="package://robotiq_description/meshes/collision/f2_140/robotiq_arg2f_${stroke}_outer_knuckle.stl" />
+          <mesh filename="package://robotiq_description/meshes/collision/2f_140/robotiq_arg2f_${stroke}_outer_knuckle.stl" />
         </geometry>
       </collision>
@@ -47,5 +47,5 @@
         <origin xyz="0 0 0" rpy="0 0 0" />
         <geometry>
-          <mesh filename="package://robotiq_description/meshes/visual/f2_140/robotiq_arg2f_${stroke}_outer_finger.stl" />
+          <mesh filename="package://robotiq_description/meshes/visual/2f_140/robotiq_arg2f_${stroke}_outer_finger.stl" />
         </geometry>
         <material name="">
@@ -56,5 +56,5 @@
         <origin xyz="0 0 0" rpy="0 0 0" />
         <geometry>
-          <mesh filename="package://robotiq_description/meshes/collision/f2_140/robotiq_arg2f_${stroke}_outer_finger.stl" />
+          <mesh filename="package://robotiq_description/meshes/collision/2f_140/robotiq_arg2f_${stroke}_outer_finger.stl" />
         </geometry>
       </collision>
@@ -77,5 +77,5 @@
         <origin xyz="0 0 0" rpy="0 0 0" />
         <geometry>
-          <mesh filename="package://robotiq_description/meshes/visual/f2_140/robotiq_arg2f_${stroke}_inner_knuckle.stl" />
+          <mesh filename="package://robotiq_description/meshes/visual/2f_140/robotiq_arg2f_${stroke}_inner_knuckle.stl" />
         </geometry>
         <material name="">
@@ -86,5 +86,5 @@
         <origin xyz="0 0 0" rpy="0 0 0" />
         <geometry>
-          <mesh filename="package://robotiq_description/meshes/collision/f2_140/robotiq_arg2f_${stroke}_inner_knuckle.stl" />
+          <mesh filename="package://robotiq_description/meshes/collision/2f_140/robotiq_arg2f_${stroke}_inner_knuckle.stl" />
         </geometry>
       </collision>
@@ -107,5 +107,5 @@
         <origin xyz="0 0 0" rpy="0 0 0" />
         <geometry>
-          <mesh filename="package://robotiq_description/meshes/visual/f2_140/robotiq_arg2f_${stroke}_inner_finger.stl" />
+          <mesh filename="package://robotiq_description/meshes/visual/2f_140/robotiq_arg2f_${stroke}_inner_finger.stl" />
         </geometry>
         <material name="">
@@ -116,5 +116,5 @@
         <origin xyz="0 0 0" rpy="0 0 0" />
         <geometry>
-          <mesh filename="package://robotiq_description/meshes/collision/f2_140/robotiq_arg2f_${stroke}_inner_finger.stl" />
+          <mesh filename="package://robotiq_description/meshes/collision/2f_140/robotiq_arg2f_${stroke}_inner_finger.stl" />
         </geometry>
       </collision>

File: robotiq_description/urdf/ur_to_robotiq_adapter.urdf.xacro (robot description, xacro)
@@ -18,5 +18,5 @@
           <origin xyz="0 0 0" rpy="0 0 0"/>
           <geometry>
-            <mesh filename="package://robotiq_description/meshes/collision/f2_85/ur_to_robotiq_adapter.stl"/>
+            <mesh filename="package://robotiq_description/meshes/collision/2f_85/ur_to_robotiq_adapter.stl"/>
           </geometry>
         </collision>

Commit message: Fix path to visual meshes for 2f_85 model

File: robotiq_description/urdf/robotiq_2f_85_macro.urdf.xacro (robot description, xacro)
@@ -27,5 +27,5 @@
             <visual>
                 <geometry>
-                    <mesh filename="file://$(find robotiq_description)/meshes/visual/robotiq_base.dae" />
+                    <mesh filename="file://$(find robotiq_description)/meshes/visual/2f_85/robotiq_base.dae" />
                 </geometry>
             </visual>
@@ -44,5 +44,5 @@
             <visual>
                 <geometry>
-                    <mesh filename="file://$(find robotiq_description)/meshes/visual/left_knuckle.dae" />
+                    <mesh filename="file://$(find robotiq_description)/meshes/visual/2f_85/left_knuckle.dae" />
                 </geometry>
             </visual>
@@ -61,5 +61,5 @@
             <visual>
                 <geometry>
-                    <mesh filename="file://$(find robotiq_description)/meshes/visual/right_knuckle.dae" />
+                    <mesh filename="file://$(find robotiq_description)/meshes/visual/2f_85/right_knuckle.dae" />
                 </geometry>
             </visual>
@@ -78,5 +78,5 @@
             <visual>
                 <geometry>
-                    <mesh filename="file://$(find robotiq_description)/meshes/visual/left_finger.dae" />
+                    <mesh filename="file://$(find robotiq_description)/meshes/visual/2f_85/left_finger.dae" />
                 </geometry>
             </visual>
@@ -95,5 +95,5 @@
             <visual>
                 <geometry>
-                    <mesh filename="file://$(find robotiq_description)/meshes/visual/right_finger.dae" />
+                    <mesh filename="file://$(find robotiq_description)/meshes/visual/2f_85/right_finger.dae" />
                 </geometry>
             </visual>
@@ -112,5 +112,5 @@
             <visual>
                 <geometry>
-                    <mesh filename="file://$(find robotiq_description)/meshes/visual/left_inner_knuckle.dae" />
+                    <mesh filename="file://$(find robotiq_description)/meshes/visual/2f_85/left_inner_knuckle.dae" />
                 </geometry>
             </visual>
@@ -129,5 +129,5 @@
             <visual>
                 <geometry>
-                    <mesh filename="file://$(find robotiq_description)/meshes/visual/right_inner_knuckle.dae" />
+                    <mesh filename="file://$(find robotiq_description)/meshes/visual/2f_85/right_inner_knuckle.dae" />
                 </geometry>
             </visual>
@@ -146,5 +146,5 @@
             <visual>
                 <geometry>
-                    <mesh filename="file://$(find robotiq_description)/meshes/visual/left_finger_tip.dae" />
+                    <mesh filename="file://$(find robotiq_description)/meshes/visual/2f_85/left_finger_tip.dae" />
                 </geometry>
             </visual>
@@ -181,5 +181,5 @@
             <visual>
                 <geometry>
-                    <mesh filename="file://$(find robotiq_description)/meshes/visual/right_finger_tip.dae" />
+                    <mesh filename="file://$(find robotiq_description)/meshes/visual/2f_85/right_finger_tip.dae" />
                 </geometry>
             </visual>

File: robotiq_description/urdf/ur_to_robotiq_adapter.urdf.xacro (robot description, xacro)
@@ -12,5 +12,5 @@
           <origin xyz="0 0 0" rpy="0 0 0" />
           <geometry>
-            <mesh filename="package://robotiq_description/meshes/visual/ur_to_robotiq_adapter.dae"/>
+            <mesh filename="package://robotiq_description/meshes/visual/2f_85/ur_to_robotiq_adapter.dae"/>
           </geometry>
         </visual>
