Commit message: Separate ignition simulation urdfs.

File: robotiq_description/urdf/gz/robotiq_gripper_macro.urdf.xacro (robot description, xacro)
@@ -1,16 +1,15 @@
 <?xml version="1.0"?>
 <robot xmlns:xacro="http://wiki.ros.org/xacro" name="robotiq_gripper">
-    <!--include macro for ros2_control-->
-    <xacro:include filename="$(find robotiq_description)/urdf/robotiq_gripper.ros2_control.xacro" />
-    <xacro:macro name="robotiq_gripper" params="parent *origin prefix com_port:=10000 use_fake_hardware:=false" >
+    <xacro:include filename="$(find robotiq_description)/urdf/gz/robotiq_gripper.ros2_control.xacro" />
+    <xacro:macro name="robotiq_gripper" params="parent *origin sim:=false prefix">
         <link name="${prefix}robotiq_85_base_link">
             <visual>
                 <geometry>
-                  <mesh filename="package://robotiq_description/meshes/visual/robotiq_base.dae" />
-                </geometry>
-            </visual>
-            <collision>
-                <geometry>
-                  <mesh filename="package://robotiq_description/meshes/collision/robotiq_base.stl" />
+                    <mesh filename="file://$(find robotiq_description)/meshes/visual/robotiq_base.dae" />
+                </geometry>
+            </visual>
+            <collision>
+                <geometry>
+                    <mesh filename="file://$(find robotiq_description)/meshes/collision/robotiq_base.stl" />
                 </geometry>
             </collision>
@@ -24,10 +23,10 @@
             <visual>
                 <geometry>
-                  <mesh filename="package://robotiq_description/meshes/visual/left_knuckle.dae" />
-                </geometry>
-            </visual>
-            <collision>
-                <geometry>
-                  <mesh filename="package://robotiq_description/meshes/collision/left_knuckle.stl" />
+                    <mesh filename="file://$(find robotiq_description)/meshes/visual/left_knuckle.dae" />
+                </geometry>
+            </visual>
+            <collision>
+                <geometry>
+                    <mesh filename="file://$(find robotiq_description)/meshes/collision/left_knuckle.stl" />
                 </geometry>
             </collision>
@@ -41,10 +40,10 @@
             <visual>
                 <geometry>
-                  <mesh filename="package://robotiq_description/meshes/visual/right_knuckle.dae" />
-                </geometry>
-            </visual>
-            <collision>
-                <geometry>
-                  <mesh filename="package://robotiq_description/meshes/collision/right_knuckle.stl" />
+                    <mesh filename="file://$(find robotiq_description)/meshes/visual/right_knuckle.dae" />
+                </geometry>
+            </visual>
+            <collision>
+                <geometry>
+                    <mesh filename="file://$(find robotiq_description)/meshes/collision/right_knuckle.stl" />
                 </geometry>
             </collision>
@@ -58,10 +57,10 @@
             <visual>
                 <geometry>
-                  <mesh filename="package://robotiq_description/meshes/visual/left_finger.dae" />
-                </geometry>
-            </visual>
-            <collision>
-                <geometry>
-                  <mesh filename="package://robotiq_description/meshes/collision/left_finger.stl" />
+                    <mesh filename="file://$(find robotiq_description)/meshes/visual/left_finger.dae" />
+                </geometry>
+            </visual>
+            <collision>
+                <geometry>
+                    <mesh filename="file://$(find robotiq_description)/meshes/collision/left_finger.stl" />
                 </geometry>
             </collision>
@@ -75,10 +74,10 @@
             <visual>
                 <geometry>
-                  <mesh filename="package://robotiq_description/meshes/visual/right_finger.dae" />
-                </geometry>
-            </visual>
-            <collision>
-                <geometry>
-                  <mesh filename="package://robotiq_description/meshes/collision/right_finger.stl" />
+                    <mesh filename="file://$(find robotiq_description)/meshes/visual/right_finger.dae" />
+                </geometry>
+            </visual>
+            <collision>
+                <geometry>
+                    <mesh filename="file://$(find robotiq_description)/meshes/collision/right_finger.stl" />
                 </geometry>
             </collision>
@@ -92,10 +91,10 @@
             <visual>
                 <geometry>
-                  <mesh filename="package://robotiq_description/meshes/visual/left_inner_knuckle.dae" />
-                </geometry>
-            </visual>
-            <collision>
-                <geometry>
-                  <mesh filename="package://robotiq_description/meshes/collision/left_inner_knuckle.stl" />
+                    <mesh filename="file://$(find robotiq_description)/meshes/visual/left_inner_knuckle.dae" />
+                </geometry>
+            </visual>
+            <collision>
+                <geometry>
+                    <mesh filename="file://$(find robotiq_description)/meshes/collision/left_inner_knuckle.stl" />
                 </geometry>
             </collision>
@@ -109,10 +108,10 @@
             <visual>
                 <geometry>
-                  <mesh filename="package://robotiq_description/meshes/visual/right_inner_knuckle.dae" />
-                </geometry>
-            </visual>
-            <collision>
-                <geometry>
-                  <mesh filename="package://robotiq_description/meshes/collision/right_inner_knuckle.stl" />
+                    <mesh filename="file://$(find robotiq_description)/meshes/visual/right_inner_knuckle.dae" />
+                </geometry>
+            </visual>
+            <collision>
+                <geometry>
+                    <mesh filename="file://$(find robotiq_description)/meshes/collision/right_inner_knuckle.stl" />
                 </geometry>
             </collision>
@@ -126,10 +125,10 @@
             <visual>
                 <geometry>
-                  <mesh filename="package://robotiq_description/meshes/visual/left_finger_tip.dae" />
-                </geometry>
-            </visual>
-            <collision>
-                <geometry>
-                  <mesh filename="package://robotiq_description/meshes/collision/left_finger_tip.stl" />
+                    <mesh filename="file://$(find robotiq_description)/meshes/visual/left_finger_tip.dae" />
+                </geometry>
+            </visual>
+            <collision>
+                <geometry>
+                    <mesh filename="file://$(find robotiq_description)/meshes/collision/left_finger_tip.stl" />
                 </geometry>
             </collision>
@@ -143,10 +142,10 @@
             <visual>
                 <geometry>
-                  <mesh filename="package://robotiq_description/meshes/visual/right_finger_tip.dae" />
-                </geometry>
-            </visual>
-            <collision>
-                <geometry>
-                  <mesh filename="package://robotiq_description/meshes/collision/right_finger_tip.stl" />
+                    <mesh filename="file://$(find robotiq_description)/meshes/visual/right_finger_tip.dae" />
+                </geometry>
+            </visual>
+            <collision>
+                <geometry>
+                    <mesh filename="file://$(find robotiq_description)/meshes/collision/right_finger_tip.stl" />
                 </geometry>
             </collision>
@@ -192,5 +191,5 @@
             <axis xyz="0 -1 0" />
             <origin xyz="0.0127 0.0 0.06142" rpy="0 0 0" />
-            <mimic joint="${prefix}robotiq_85_left_knuckle_joint" />
+            <mimic joint="robotiq_85_left_knuckle_joint" />
         </joint>
         <joint name="${prefix}robotiq_85_right_inner_knuckle_joint" type="continuous">
@@ -199,5 +198,5 @@
             <axis xyz="0 -1 0" />
             <origin xyz="-0.0127 0.0 0.06142" rpy="0 0 0" />
-            <mimic joint="${prefix}robotiq_85_left_knuckle_joint" multiplier="-1" />
+            <mimic joint="robotiq_85_left_knuckle_joint" multiplier="-1" />
         </joint>
         <joint name="${prefix}robotiq_85_left_finger_tip_joint" type="continuous">
@@ -206,5 +205,5 @@
             <axis xyz="0 -1 0" />
             <origin xyz="0.00563134 0.0 0.04718515" rpy="0 0 0" />
-            <mimic joint="${prefix}robotiq_85_left_knuckle_joint" multiplier="-1" />
+            <mimic joint="robotiq_85_left_knuckle_joint" multiplier="-1" />
         </joint>
         <joint name="${prefix}robotiq_85_right_finger_tip_joint" type="continuous">
@@ -213,11 +212,7 @@
             <axis xyz="0 -1 0" />
             <origin xyz="-0.00563134 0.0 0.04718515" rpy="0 0 0" />
-            <mimic joint="${prefix}robotiq_85_left_knuckle_joint" />
-        </joint>
-        <!--instance of robotiq ros2 control hardware interface-->
-        <xacro:robotiq_gripper_ros2_control
-          name="${prefix}robotiq_gripper_hardware_interface"
-          use_fake_hardware="${use_fake_hardware}"
-          com_port="${com_port}"/>
+            <mimic joint="robotiq_85_left_knuckle_joint" />
+        </joint>
+        <xacro:robotiq_gz_gripper_ros2_control name="IgnitionSystem"/>
     </xacro:macro>
 </robot>

File: robotiq_description/urdf/robotiq_gripper.ros2_control.xacro (robot description, xacro)
@@ -1,7 +1,7 @@
 <?xml version="1.0"?>
 <robot xmlns:xacro="http://www.ros.org/wiki/xacro">
-    <xacro:macro name="robotiq_gripper_ros2_control" params="name com_port use_fake_hardware:=false sim_gz:=false">
+    <xacro:macro name="robotiq_gripper_ros2_control" params="name com_port use_fake_hardware:=false">
         <!-- ros2_control custom hardware interface -->
-        <xacro:unless value="${use_fake_hardware or sim_gz}">
+        <xacro:unless value="${use_fake_hardware}">
             <ros2_control name="${name}" type="actuator">
                 <hardware>
@@ -20,15 +20,9 @@
             </ros2_control>
         </xacro:unless>
-        <xacro:if value="${use_fake_hardware or sim_gz}">
+        <xacro:if value="${use_fake_hardware}">
             <ros2_control name="${name}" type="system">
                 <hardware>
                     <!-- ros2_control fake component -->
-                    <xacro:if value="${use_fake_hardware}">
-                        <plugin>fake_components/GenericSystem</plugin>
-                    </xacro:if>
-                    <!-- gz simulation -->
-                    <xacro:if value="${sim_gz}">
-                        <plugin>ign_ros2_control/IgnitionSystem</plugin>
-                    </xacro:if>
+                    <plugin>fake_components/GenericSystem</plugin>
                 </hardware>
                 <joint name="robotiq_85_left_knuckle_joint">
@@ -74,12 +68,4 @@
                 </joint>
             </ros2_control>
-            <!--gz plugin for ros2 control -->
-            <xacro:if value="${sim_gz}">
-                <gazebo>
-                    <plugin filename="ign_ros2_control-system" name="ign_ros2_control::IgnitionROS2ControlPlugin">
-                        <parameters>$(find robotiq_driver)/config/robotiq_controllers.yaml</parameters>
-                    </plugin>
-                </gazebo>
-            </xacro:if>
         </xacro:if>
     </xacro:macro>

File: robotiq_description/urdf/robotiq_gripper.urdf.xacro (robot description, xacro)
@@ -4,5 +4,4 @@
     <xacro:arg name="com_port" default="10000" />
     <xacro:arg name="use_fake_hardware" default="false" />
-    <xacro:arg name="sim_gz" default="true" />
     <!-- Import macros -->
     <xacro:include filename="$(find robotiq_description)/urdf/robotiq_gripper_macro.urdf.xacro" />
@@ -11,5 +10,4 @@
       parent="world"
       use_fake_hardware="$(arg use_fake_hardware)"
-      sim_gz="$(arg sim_gz)"
       com_port="$(arg com_port)"
       prefix="">
