Commit message: Remove publishing of mimic joints. Reorganize sim urdfs.

File: robotiq_description/urdf/gz/robotiq_gripper.ros2_control.xacro (robot description, xacro)
@@ -17,35 +17,20 @@
                 <param name="mimic">robotiq_85_left_knuckle_joint</param>
                 <param name="multiplier">-1</param>
-                <command_interface name="position"/>
-                <state_interface name="position"/>
-                <state_interface name="velocity"/>
             </joint>
             <joint name="robotiq_85_left_inner_knuckle_joint">
                 <param name="mimic">robotiq_85_left_knuckle_joint</param>
                 <param name="multiplier">1</param>
-                <command_interface name="position" />
-                <state_interface name="position" />
-                <state_interface name="velocity" />
             </joint>
             <joint name="robotiq_85_right_inner_knuckle_joint">
                 <param name="mimic">robotiq_85_left_knuckle_joint</param>
                 <param name="multiplier">-1</param>
-                <command_interface name="position" />
-                <state_interface name="position" />
-                <state_interface name="velocity" />
             </joint>
             <joint name="robotiq_85_left_finger_tip_joint">
                 <param name="mimic">robotiq_85_left_knuckle_joint</param>
                 <param name="multiplier">-1</param>
-                <command_interface name="position" />
-                <state_interface name="position" />
-                <state_interface name="velocity" />
             </joint>
             <joint name="robotiq_85_right_finger_tip_joint">
                 <param name="mimic">robotiq_85_left_knuckle_joint</param>
                 <param name="multiplier">1</param>
-                <command_interface name="position" />
-                <state_interface name="position" />
-                <state_interface name="velocity" />
             </joint>
         </ros2_control>

File: robotiq_description/urdf/gz/robotiq_gripper.urdf.xacro (robot description, xacro)
@@ -2,4 +2,5 @@
 <robot xmlns:xacro="http://wiki.ros.org/xacro" name="robotiq_gripper">
     <!-- Import macros -->
+    <xacro:include filename="$(find robotiq_description)/urdf/gz/robotiq_gripper.ros2_control.xacro" />
     <xacro:include filename="$(find robotiq_description)/urdf/gz/robotiq_gripper_macro.urdf.xacro" />
     <link name="world" />
@@ -9,4 +10,5 @@
         <origin xyz="0 0 0" rpy="0 0 0" />
     </xacro:robotiq_gripper>
+    <xacro:robotiq_gz_gripper_ros2_control name="IgnitionSystem"/>
     <gazebo>
         <plugin filename="ign_ros2_control-system" name="ign_ros2_control::IgnitionROS2ControlPlugin">

File: robotiq_description/urdf/gz/robotiq_gripper_macro.urdf.xacro (robot description, xacro)
@@ -1,6 +1,5 @@
 <?xml version="1.0"?>
 <robot xmlns:xacro="http://wiki.ros.org/xacro" name="robotiq_gripper">
-    <xacro:include filename="$(find robotiq_description)/urdf/gz/robotiq_gripper.ros2_control.xacro" />
-    <xacro:macro name="robotiq_gripper" params="parent *origin sim:=false prefix">
+    <xacro:macro name="robotiq_gripper" params="parent *origin prefix">
         <link name="${prefix}robotiq_85_base_link">
             <visual>
@@ -214,5 +213,4 @@
             <mimic joint="robotiq_85_left_knuckle_joint" />
         </joint>
-        <xacro:robotiq_gz_gripper_ros2_control name="IgnitionSystem"/>
     </xacro:macro>
 </robot>
